File: PCB/Right/Pragmatic.sch (KiCad schematic (older format))
At the start: 75 parts, among them J1 Conn_02x07_Odd_Even, SW1 SW_Push, SW10 SW_Push, SW11 SW_Push, SW12 SW_Push, SW13 SW_Push, SW14 SW_Push, SW15 SW_Push, SW16 SW_Push, SW17 SW_Push, SW18 SW_Push, SW19 SW_Push, SW2 SW_Push, SW20 SW_Push, SW21 SW_Push, SW22 SW_Push, SW23 SW_Push, SW24 SW_Push, SW25 SW_Push, SW26 SW_Push, SW27 SW_Push, SW28 SW_Push, SW29 SW_Push, SW3 SW_Push, SW30 SW_Push, SW31 SW_Push, SW32 SW_Push, SW33 SW_Push, SW34 SW_Push, SW35 SW_Push, SW36 SW_Push, SW4 SW_Push, SW5 SW_Push, SW6 SW_Push, SW7 SW_Push, SW8 SW_Push, SW9 SW_Push

Commit message: right
Connections:
- net Col10: now also SW10.2, SW16.2, SW22.2, SW28.2, SW34.2, SW4.2; no longer SW15.2, SW21.2, SW27.2, SW3.2, SW33.2, SW9.2
- net Col11: now also SW11.2, SW17.2, SW23.2, SW29.2, SW35.2, SW5.2; no longer SW14.2, SW2.2, SW20.2, SW26.2, SW32.2, SW8.2
- net Col12: now also SW12.2, SW18.2, SW24.2, SW30.2, SW36.2, SW6.2; no longer SW1.2, SW13.2, SW19.2, SW25.2, SW31.2, SW7.2
- net Col7: now also SW1.2, SW13.2, SW19.2, SW25.2, SW31.2, SW7.2; no longer SW12.2, SW18.2, SW24.2, SW30.2, SW36.2, SW6.2
- net Col8: now also SW14.2, SW2.2, SW20.2, SW26.2, SW32.2, SW8.2; no longer SW11.2, SW17.2, SW23.2, SW29.2, SW35.2, SW5.2
- net Col9: now also SW15.2, SW21.2, SW27.2, SW3.2, SW33.2, SW9.2; no longer SW10.2, SW16.2, SW22.2, SW28.2, SW34.2, SW4.2
Changed lines of the file:
@@
 Wire Wire Line
 	4900 2700 4900 3000
-Text GLabel 4900 2700 1    50   Input ~ 0
+Text GLabel 2400 2700 1    50   Input ~ 0
 Col7
 Wire Wire Line
@@
 Wire Wire Line
 	5700 4100 5700 4200
-Text GLabel 2400 2700 1    50   Input ~ 0
+Text GLabel 4900 2700 1    50   Input ~ 0
 Col12
+Text GLabel 4400 2700 1    50   Input ~ 0
+Col11
+Text GLabel 3900 2700 1    50   Input ~ 0
+Col10
+Text GLabel 3400 2700 1    50   Input ~ 0
+Col9
 Text GLabel 2900 2700 1    50   Input ~ 0
-Col11
-Text GLabel 3400 2700 1    50   Input ~ 0
-Col10
-Text GLabel 3900 2700 1    50   Input ~ 0
-Col9
-Text GLabel 4400 2700 1    50   Input ~ 0
 Col8
 $EndSCHEMATC

Commit message: finish up
Connections:
- wire segments 77 -> 79
Other:
- moved on the sheet: D37, R1
Changed lines of the file:
@@
 L Device:LED D37
 U 1 1 619DFFCE
+P 5700 4350
+F 0 "D37" V 5600 4450 50  0000 L CNN
+F 1 "LED" V 5700 4450 50  0000 L CNN
+F 2 "LED_THT:LED_D3.0mm" H 5700 4350 50  0001 C CNN
+F 3 "~" H 5700 4350 50  0001 C CNN
+	1    5700 4350
+	0    -1   -1   0
+$EndComp
+$Comp
+L Device:R R1
+U 1 1 619DF3E5
 P 5700 3950
-F 0 "D37" V 5600 4050 50  0000 L CNN
-F 1 "LED" V 5700 4050 50  0000 L CNN
-F 2 "LED_THT:LED_D3.0mm" H 5700 3950 50  0001 C CNN
+F 0 "R1" H 5800 4000 50  0000 L CNN
+F 1 "220Ω" H 5800 3950 50  0000 L CNN
+F 2 "Resistor_THT:R_Axial_DIN0207_L6.3mm_D2.5mm_P10.16mm_Horizontal" V 5630 3950 50  0001 C CNN
 F 3 "~" H 5700 3950 50  0001 C CNN
 	1    5700 3950
-	0    1    1    0
-$EndComp
-$Comp
-L Device:R R1
-U 1 1 619DF3E5
-P 5700 4350
-F 0 "R1" H 5800 4400 50  0000 L CNN
-F 1 "220Ω" H 5800 4350 50  0000 L CNN
-F 2 "Resistor_THT:R_Axial_DIN0207_L6.3mm_D2.5mm_P10.16mm_Horizontal" V 5630 4350 50  0001 C CNN
-F 3 "~" H 5700 4350 50  0001 C CNN
-	1    5700 4350
-	1    0    0    -1
+	-1   0    0    1
 $EndComp
 Wire Wire Line
@@
 	6800 3200 6800 3300
 Wire Wire Line
-	5700 4100 5700 4200
+	5700 4200 5700 4100
 Text GLabel 4900 2700 1    50   Input ~ 0
 Col12
@@
 Text GLabel 2900 2700 1    50   Input ~ 0
 Col8
+$Comp
+L power:PWR_FLAG #FLG0101
+U 1 1 61885ADD
+P 7150 2500
+F 0 "#FLG0101" H 7150 2575 50  0001 C CNN
+F 1 "PWR_FLAG" H 7150 2673 50  0000 C CNN
+F 2 "" H 7150 2500 50  0001 C CNN
+F 3 "~" H 7150 2500 50  0001 C CNN
+	1    7150 2500
+	1    0    0    -1
+$EndComp
+$Comp
+L power:PWR_FLAG #FLG0102
+U 1 1 61886641
+P 7150 3300
+F 0 "#FLG0102" H 7150 3375 50  0001 C CNN
+F 1 "PWR_FLAG" H 7150 3473 50  0000 C CNN
+F 2 "" H 7150 3300 50  0001 C CNN
+F 3 "~" H 7150 3300 50  0001 C CNN
+	1    7150 3300
+	1    0    0    -1
+$EndComp
+Wire Wire Line
+	7150 3300 6800 3300
+Connection ~ 6800 3300
+Wire Wire Line
+	7150 2500 6800 2500
+Connection ~ 6800 2500
 $EndSCHEMATC
