File: PCB/Hand/Pragmatic.sch (KiCad schematic (older format))
At the start: 76 parts, among them J1 Conn_02x08_Odd_Even, J2 Conn_01x04, SW1 SW_Push, SW10 SW_Push, SW11 SW_Push, SW12 SW_Push, SW13 SW_Push, SW14 SW_Push, SW15 SW_Push, SW16 SW_Push, SW17 SW_Push, SW18 SW_Push, SW19 SW_Push, SW2 SW_Push, SW20 SW_Push, SW21 SW_Push, SW22 SW_Push, SW23 SW_Push, SW24 SW_Push, SW25 SW_Push, SW26 SW_Push, SW27 SW_Push, SW28 SW_Push, SW29 SW_Push, SW3 SW_Push, SW30 SW_Push, SW31 SW_Push, SW32 SW_Push, SW33 SW_Push, SW34 SW_Push, SW35 SW_Push, SW36 SW_Push, SW4 SW_Push, SW5 SW_Push, SW6 SW_Push, SW7 SW_Push, SW8 SW_Push, SW9 SW_Push

Commit message: double side design
Parts:
- D1, D10, D11, D12, D13, D14, D15, D16, D17, D18, D19, D2, D20, D21, D22, D23, D24, D25, D26, D27, D28, D29, D3, D30, D31, D32, D33, D34, D35, D36, D4, D5, D6, D7, D8, D9: footprint Pragmatic:D_SMD -> Pragmatic:D_SMD_With_Shadow; LCSC (none) -> C81598
- D37: footprint LED_SMD:LED_0805_2012Metric_Pad1.15x1.40mm_HandSolder -> Pragmatic:LED_0805_With_Shadow; LCSC (none) -> C2297
- J1: LCSC (none) -> C3406
- R1: value 220Ω -> R; footprint Resistor_SMD:R_0805_2012Metric_Pad1.20x1.40mm_HandSolder -> Pragmatic:R_0805_With_Shadow; LCSC (none) -> C17408
- SW1, SW10, SW11, SW12, SW13, SW14, SW15, SW16, SW17, SW18, SW19, SW2, SW20, SW21, SW22, SW23, SW24, SW25, SW26, SW27, SW28, SW29, SW3, SW30, SW31, SW32, SW33, SW34, SW35, SW36, SW4, SW5, SW6, SW7, SW8, SW9: footprint Pragmatic:CherryMX_ChocV2_1u -> Pragmatic:Switch_1u_Mirrored
Connections:
- net +5V: now also R1.1; no longer R1.2
- net at D37.2 (A): now also R1.2; no longer R1.1
Other:
- moved on the sheet: J2

Commit message: left hand done.
Parts:
- J2: footprint kbd:OLED -> Connector_PinHeader_2.54mm:PinHeader_1x04_P2.54mm_Vertical
Changed lines of the file:
@@
 F 0 "J2" H 7418 2825 50  0000 C CNN
 F 1 "Conn_01x04" H 7418 2916 50  0000 C CNN
-F 2 "kbd:OLED" H 7500 3250 50  0001 C CNN
+F 2 "Connector_PinHeader_2.54mm:PinHeader_1x04_P2.54mm_Vertical" H 7500 3250 50  0001 C CNN
 F 3 "~" H 7500 3250 50  0001 C CNN
 	1    7500 3250

Commit message: details
Parts:
- added H1, H2, H3, H4: MountingHole, MountingHole:MountingHole_3.2mm_M3_DIN965_Pad_TopBottom, symbol Mechanical:MountingHole
- J1: footprint Connector_IDC:IDC-Header_2x08_P2.54mm_Vertical -> Pragmatic:IDC-Header_2x08_P2.54mm_Vertical_Mirrored
- J2: footprint Connector_PinHeader_2.54mm:PinHeader_1x04_P2.54mm_Vertical -> Connector_PinSocket_2.54mm:PinSocket_1x04_P2.54mm_Vertical
- SW14: value SW_Push -> Q
- SW15: value SW_Push -> W
- SW16: value SW_Push -> E
- SW17: value SW_Push -> R
- SW18: value SW_Push -> T
- SW20: value SW_Push -> A
- SW21: value SW_Push -> S
- SW22: value SW_Push -> D
- SW23: value SW_Push -> F
- SW24: value SW_Push -> G
- SW26: value SW_Push -> Z
- SW27: value SW_Push -> X
- SW28: value SW_Push -> C
- SW29: value SW_Push -> V
- SW30: value SW_Push -> B
Changed lines of the file:
@@
 P 4700 5400
 F 0 "SW30" H 4700 5593 50  0000 C CNN
-F 1 "SW_Push" H 4700 5594 50  0001 C CNN
+F 1 "B" H 4700 5594 50  0001 C CNN
 F 2 "Pragmatic:Switch_1u_Mirrored" H 4700 5600 50  0001 C CNN
 F 3 "~" H 4700 5600 50  0001 C CNN
@@
 P 4200 5400
 F 0 "SW29" H 4200 5593 50  0000 C CNN
-F 1 "SW_Push" H 4200 5594 50  0001 C CNN
+F 1 "V" H 4200 5594 50  0001 C CNN
 F 2 "Pragmatic:Switch_1u_Mirrored" H 4200 5600 50  0001 C CNN
 F 3 "~" H 4200 5600 50  0001 C CNN
@@
 P 3700 5400
 F 0 "SW28" H 3700 5593 50  0000 C CNN
-F 1 "SW_Push" H 3700 5594 50  0001 C CNN
+F 1 "C" H 3700 5594 50  0001 C CNN
 F 2 "Pragmatic:Switch_1u_Mirrored" H 3700 5600 50  0001 C CNN
 F 3 "~" H 3700 5600 50  0001 C CNN
@@
 P 3200 5400
 F 0 "SW27" H 3200 5593 50  0000 C CNN
-F 1 "SW_Push" H 3200 5594 50  0001 C CNN
+F 1 "X" H 3200 5594 50  0001 C CNN
 F 2 "Pragmatic:Switch_1u_Mirrored" H 3200 5600 50  0001 C CNN
 F 3 "~" H 3200 5600 50  0001 C CNN
@@
 P 2700 5400
 F 0 "SW26" H 2700 5593 50  0000 C CNN
-F 1 "SW_Push" H 2700 5594 50  0001 C CNN
+F 1 "Z" H 2700 5594 50  0001 C CNN
 F 2 "Pragmatic:Switch_1u_Mirrored" H 2700 5600 50  0001 C CNN
 F 3 "~" H 2700 5600 50  0001 C CNN
@@
 P 4700 4800
 F 0 "SW24" H 4700 4993 50  0000 C CNN
-F 1 "SW_Push" H 4700 4994 50  0001 C CNN
+F 1 "G" H 4700 4994 50  0001 C CNN
 F 2 "Pragmatic:Switch_1u_Mirrored" H 4700 5000 50  0001 C CNN
 F 3 "~" H 4700 5000 50  0001 C CNN
@@
 P 4200 4800
 F 0 "SW23" H 4200 4993 50  0000 C CNN
-F 1 "SW_Push" H 4200 4994 50  0001 C CNN
+F 1 "F" H 4200 4994 50  0001 C CNN
 F 2 "Pragmatic:Switch_1u_Mirrored" H 4200 5000 50  0001 C CNN
 F 3 "~" H 4200 5000 50  0001 C CNN
@@
 P 3700 4800
 F 0 "SW22" H 3700 4993 50  0000 C CNN
-F 1 "SW_Push" H 3700 4994 50  0001 C CNN
+F 1 "D" H 3700 4994 50  0001 C CNN
 F 2 "Pragmatic:Switch_1u_Mirrored" H 3700 5000 50  0001 C CNN
 F 3 "~" H 3700 5000 50  0001 C CNN
@@
 P 3200 4800
 F 0 "SW21" H 3200 4993 50  0000 C CNN
-F 1 "SW_Push" H 3200 4994 50  0001 C CNN
+F 1 "S" H 3200 4994 50  0001 C CNN
 F 2 "Pragmatic:Switch_1u_Mirrored" H 3200 5000 50  0001 C CNN
 F 3 "~" H 3200 5000 50  0001 C CNN
@@
 $EndComp
 $Comp
-L Switch:SW_Push SW20
-U 1 1 618C1817
-P 2700 4800
-F 0 "SW20" H 2700 4993 50  0000 C CNN
-F 1 "SW_Push" H 2700 4994 50  0001 C CNN
-F 2 "Pragmatic:Switch_1u_Mirrored" H 2700 5000 50  0001 C CNN
-F 3 "~" H 2700 5000 50  0001 C CNN
-	1    2700 4800
-	1    0    0    -1
-$EndComp
-$Comp
 L Device:D D20
 U 1 1 618C1811
@@
 P 4700 4200
 F 0 "SW18" H 4700 4393 50  0000 C CNN
-F 1 "SW_Push" H 4700 4394 50  0001 C CNN
+F 1 "T" H 4700 4394 50  0001 C CNN
 F 2 "Pragmatic:Switch_1u_Mirrored" H 4700 4400 50  0001 C CNN
 F 3 "~" H 4700 4400 50  0001 C CNN
@@
 P 4200 4200
 F 0 "SW17" H 4200 4393 50  0000 C CNN
-F 1 "SW_Push" H 4200 4394 50  0001 C CNN
+F 1 "R" H 4200 4394 50  0001 C CNN
 F 2 "Pragmatic:Switch_1u_Mirrored" H 4200 4400 50  0001 C CNN
 F 3 "~" H 4200 4400 50  0001 C CNN
@@
 P 3700 4200
 F 0 "SW16" H 3700 4393 50  0000 C CNN
-F 1 "SW_Push" H 3700 4394 50  0001 C CNN
+F 1 "E" H 3700 4394 50  0001 C CNN
 F 2 "Pragmatic:Switch_1u_Mirrored" H 3700 4400 50  0001 C CNN
 F 3 "~" H 3700 4400 50  0001 C CNN
@@
 P 3200 4200
 F 0 "SW15" H 3200 4393 50  0000 C CNN
-F 1 "SW_Push" H 3200 4394 50  0001 C CNN
+F 1 "W" H 3200 4394 50  0001 C CNN
 F 2 "Pragmatic:Switch_1u_Mirrored" H 3200 4400 50  0001 C CNN
 F 3 "~" H 3200 4400 50  0001 C CNN
@@
 P 2700 4200
 F 0 "SW14" H 2700 4393 50  0000 C CNN
-F 1 "SW_Push" H 2700 4394 50  0001 C CNN
+F 1 "Q" H 2700 4394 50  0001 C CNN
 F 2 "Pragmatic:Switch_1u_Mirrored" H 2700 4400 50  0001 C CNN
 F 3 "~" H 2700 4400 50  0001 C CNN
@@
 F 0 "J1" H 6000 3367 50  0000 C CNN
 F 1 "Conn_02x08_Odd_Even" H 6000 3276 50  0000 C CNN
-F 2 "Connector_IDC:IDC-Header_2x08_P2.54mm_Vertical" H 5950 2850 50  0001 C CNN
+F 2 "Pragmatic:IDC-Header_2x08_P2.54mm_Vertical_Mirrored" H 5950 2850 50  0001 C CNN
 F 3 "~" H 5950 2850 50  0001 C CNN
 F 4 "C3406" H 5950 2850 50  0001 C CNN "LCSC"
@@
 F 0 "J2" H 7418 2825 50  0000 C CNN
 F 1 "Conn_01x04" H 7418 2916 50  0000 C CNN
-F 2 "Connector_PinHeader_2.54mm:PinHeader_1x04_P2.54mm_Vertical" H 7500 3250 50  0001 C CNN
+F 2 "Connector_PinSocket_2.54mm:PinSocket_1x04_P2.54mm_Vertical" H 7500 3250 50  0001 C CNN
 F 3 "~" H 7500 3250 50  0001 C CNN
 	1    7500 3250
@@
 Wire Wire Line
 	5950 5250 6200 5250
+$Comp
+L Switch:SW_Push SW20
+U 1 1 618C1817
+P 2700 4800
+F 0 "SW20" H 2700 4993 50  0000 C CNN
+F 1 "A" H 2700 4994 50  0001 C CNN
+F 2 "Pragmatic:Switch_1u_Mirrored" H 2700 5000 50  0001 C CNN
+F 3 "~" H 2700 5000 50  0001 C CNN
+	1    2700 4800
+	1    0    0    -1
+$EndComp
+$Comp
+L Mechanical:MountingHole H1
+U 1 1 61BDFA75
+P 6850 3950
+F 0 "H1" H 6950 3996 50  0000 L CNN
+F 1 "MountingHole" H 6950 3905 50  0000 L CNN
+F 2 "MountingHole:MountingHole_3.2mm_M3_DIN965_Pad_TopBottom" H 6850 3950 50  0001 C CNN
+F 3 "~" H 6850 3950 50  0001 C CNN
+	1    6850 3950
+	1    0    0    -1
+$EndComp
+$Comp
+L Mechanical:MountingHole H2
+U 1 1 61BE2378
+P 6850 4200
+F 0 "H2" H 6950 4246 50  0000 L CNN
+F 1 "MountingHole" H 6950 4155 50  0000 L CNN
+F 2 "MountingHole:MountingHole_3.2mm_M3_DIN965_Pad_TopBottom" H 6850 4200 50  0001 C CNN
+F 3 "~" H 6850 4200 50  0001 C CNN
+	1    6850 4200
+	1    0    0    -1
+$EndComp
+$Comp
+L Mechanical:MountingHole H3
+U 1 1 61BE27F5
+P 6850 4450
+F 0 "H3" H 6950 4496 50  0000 L CNN
+F 1 "MountingHole" H 6950 4405 50  0000 L CNN
+F 2 "MountingHole:MountingHole_3.2mm_M3_DIN965_Pad_TopBottom" H 6850 4450 50  0001 C CNN
+F 3 "~" H 6850 4450 50  0001 C CNN
+	1    6850 4450
+	1    0    0    -1
+$EndComp
+$Comp
+L Mechanical:MountingHole H4
+U 1 1 61BE2BA9
+P 6850 4700
+F 0 "H4" H 6950 4746 50  0000 L CNN
+F 1 "MountingHole" H 6950 4655 50  0000 L CNN
+F 2 "MountingHole:MountingHole_3.2mm_M3_DIN965_Pad_TopBottom" H 6850 4700 50  0001 C CNN
+F 3 "~" H 6850 4700 50  0001 C CNN
+	1    6850 4700
+	1    0    0    -1
+$EndComp
 $EndSCHEMATC

Commit message: controller done
Connections:
- net +5V: now also J1.2 (Pin_2); no longer J1.1 (Pin_1)
- net Col1: now also J1.5 (Pin_5); no longer J1.6 (Pin_6)
- net Col2: now also J1.7 (Pin_7); no longer J1.8 (Pin_8)
- net Col3: now also J1.9 (Pin_9); no longer J1.10 (Pin_10)
- net Col4: now also J1.11 (Pin_11); no longer J1.12 (Pin_12)
- net Col5: now also J1.13 (Pin_13); no longer J1.14 (Pin_14)
- net Col6: now also J1.15 (Pin_15); no longer J1.16 (Pin_16)
- net GND: now also J1.1 (Pin_1); no longer J1.2 (Pin_2)
- net Row1: now also J1.6 (Pin_6); no longer J1.5 (Pin_5)
- net Row2: now also J1.8 (Pin_8); no longer J1.7 (Pin_7)
- net Row3: now also J1.10 (Pin_10); no longer J1.9 (Pin_9)
- net Row4: now also J1.12 (Pin_12); no longer J1.11 (Pin_11)
- net Row5: now also J1.14 (Pin_14); no longer J1.13 (Pin_13)
- net Row6: now also J1.16 (Pin_16); no longer J1.15 (Pin_15)
Changed lines of the file:
@@
 	10550 4050 10150 4050
 Connection ~ 10150 4050
+Text GLabel 6250 2550 2    50   Input ~ 0
+VCC
 Text GLabel 5750 2550 0    50   Input ~ 0
-VCC
-Text GLabel 6250 2550 2    50   Input ~ 0
 GND
 Text GLabel 6250 2650 2    50   Input ~ 0
@@
 Text GLabel 5750 2650 0    50   Input ~ 0
 SCL
-Text GLabel 5750 2750 0    50   Input ~ 0
+Text GLabel 6250 2750 2    50   Input ~ 0
 Row1
+Text GLabel 6250 2850 2    50   Input ~ 0
+Row2
+Text GLabel 6250 2950 2    50   Input ~ 0
+Row3
+Text GLabel 6250 3050 2    50   Input ~ 0
+Row4
+Text GLabel 6250 3150 2    50   Input ~ 0
+Row5
+Text GLabel 6250 3250 2    50   Input ~ 0
+Row6
 Text GLabel 5750 2850 0    50   Input ~ 0
-Row2
+Col2
 Text GLabel 5750 2950 0    50   Input ~ 0
-Row3
+Col3
 Text GLabel 5750 3050 0    50   Input ~ 0
-Row4
-Text GLabel 5750 3150 0    50   Input ~ 0
-Row5
+Col4
 Text GLabel 5750 3250 0    50   Input ~ 0
-Row6
-Text GLabel 6250 2750 2    50   Input ~ 0
-Col1
-Text GLabel 6250 2850 2    50   Input ~ 0
-Col2
-Text GLabel 6250 2950 2    50   Input ~ 0
-Col3
-Text GLabel 6250 3050 2    50   Input ~ 0
-Col4
-Text GLabel 6250 3150 2    50   Input ~ 0
-Col5
-Text GLabel 6250 3250 2    50   Input ~ 0
 Col6
 Text GLabel 7700 3050 2    50   Input ~ 0
@@
 Text GLabel 7700 3150 2    50   Input ~ 0
 VCC
-$Comp
-L Connector_Generic:Conn_02x08_Odd_Even J1
-U 1 1 6194905D
-P 5950 2850
-F 0 "J1" H 6000 3367 50  0000 C CNN
-F 1 "Conn_02x08_Odd_Even" H 6000 3276 50  0000 C CNN
-F 2 "Pragmatic:IDC-Header_2x08_P2.54mm_Vertical_Mirrored" H 5950 2850 50  0001 C CNN
-F 3 "~" H 5950 2850 50  0001 C CNN
-F 4 "C3406" H 5950 2850 50  0001 C CNN "LCSC"
-	1    5950 2850
-	1    0    0    -1
-$EndComp
 $Comp
 L Connector_Generic:Conn_01x04 J2
@@
 	1    0    0    -1
 $EndComp
+$Comp
+L Connector_Generic:Conn_02x08_Odd_Even J1
+U 1 1 6194905D
+P 5950 2850
+F 0 "J1" H 6000 3367 50  0000 C CNN
+F 1 "Conn_02x08_Odd_Even" H 6000 3276 50  0000 C CNN
+F 2 "Pragmatic:IDC-Header_2x08_P2.54mm_Vertical_Mirrored" H 5950 2850 50  0001 C CNN
+F 3 "~" H 5950 2850 50  0001 C CNN
+F 4 "C3406" H 5950 2850 50  0001 C CNN "LCSC"
+	1    5950 2850
+	1    0    0    -1
+$EndComp
+Text GLabel 5750 2750 0    50   Input ~ 0
+Col1
+Text GLabel 5750 3150 0    50   Input ~ 0
+Col5
 $EndSCHEMATC
