File: PCB/V1/Control/Pragmatic.kicad_sch (KiCad schematic)
At the start: 4 parts, among them J1 L, J2 R, SW1 SW_Push, U1 ProMicro

Commit message: v2
Parts:
- added J3: Conn_01x04, Connector_PinSocket_2.54mm:PinSocket_1x04_P2.54mm_Vertical, symbol Connector_Generic:Conn_01x04
Connections:
- net +5V: now also J1.2 (Pin_2), J3.3 (Pin_3); no longer J1.1 (Pin_1)
- net Col1: now also J1.3 (Pin_3); no longer J1.4 (Pin_4)
- net Col10: now also J2.8 (Pin_8); no longer J2.10 (Pin_10)
- net Col11: now also J2.6 (Pin_6); no longer J2.12 (Pin_12)
- net Col12: now also J2.4 (Pin_4); no longer J2.14 (Pin_14)
- net Col2: now also J1.5 (Pin_5); no longer J1.6 (Pin_6)
- net Col3: now also J1.7 (Pin_7); no longer J1.8 (Pin_8)
- net Col4: now also J1.9 (Pin_9); no longer J1.10 (Pin_10)
- net Col5: now also J1.11 (Pin_11); no longer J1.12 (Pin_12)
- net Col6: now also J1.13 (Pin_13); no longer J1.14 (Pin_14)
- net Col7: now also J2.14 (Pin_14); no longer J2.4 (Pin_4)
- net Col8: now also J2.12 (Pin_12); no longer J2.6 (Pin_6)
- net Col9: now also J2.10 (Pin_10); no longer J2.8 (Pin_8)
- net GND: now also J1.1 (Pin_1), J3.4 (Pin_4); no longer J1.2 (Pin_2)
- net Row1: now also J1.4 (Pin_4), J3.1 (Pin_1); no longer J1.3 (Pin_3)
- net Row2: now also J1.6 (Pin_6), J3.2 (Pin_2); no longer J1.5 (Pin_5)
- net Row3: now also J1.8 (Pin_8); no longer J1.7 (Pin_7)
- net Row4: now also J1.10 (Pin_10); no longer J1.9 (Pin_9)
- net Row5: now also J1.12 (Pin_12); no longer J1.11 (Pin_11)
- net Row6: now also J1.14 (Pin_14); no longer J1.13 (Pin_13)
