File: PCB/Input Hotswap/Pragmatic.kicad_pcb (KiCad board)
At the start: 2 copper layers, 114.3 x 127 mm, 82 parts, among them J1 Hand-Soldering, SW1 SW_Push, SW10 SW_Push, SW11 SW_Push, SW12 SW_Push, SW13 SW_Push, SW14 SW_Push, SW15 SW_Push, SW16 SW_Push, SW17 SW_Push, SW18 SW_Push, SW19 SW_Push, SW2 SW_Push, SW20 SW_Push, SW21 SW_Push, SW22 SW_Push, SW23 SW_Push, SW24 SW_Push, SW25 SW_Push, SW26 SW_Push, SW27 SW_Push, SW28 SW_Push, SW29 SW_Push, SW3 SW_Push, SW30 SW_Push, SW31 SW_Push, SW32 SW_Push, SW33 SW_Push, SW34 SW_Push, SW35 SW_Push, SW36 SW_Push, SW4 SW_Push, SW5 SW_Push, SW6 SW_Push, SW7 SW_Push, SW8 SW_Push, SW9 SW_Push

Commit message: v2
Other:
- board text added: "6X6 input module designed by James Sa https://github.com/jamessa/Pragmatic"
- board text added: "V2.1 Hotswap"
- board text removed: "6X6 input module designed by James Sa"
- board text removed: "Bart"
- board text removed: "NeweFre"
- board text removed: "SJ"
- board text removed: "V2 Hotswap"
- board text removed: "務實鍵盤2022"
- board text removed: "我噠噠的敲擊聲，是歸人，是過客，是靈思泉湧時短暫殘留的腳印。"
- board text removed: "棠。"
- board text removed: "王證淇"
- board text removed: "誰知PCB，片片皆辛苦。"
