File: PCB/Plate/Plate.kicad_pcb (KiCad board)
At the start: 2 copper layers, 114.3 x 114.3 mm, 43 parts

Commit message: v2
Parts:
- removed the REF** at (127.0, 135.3)
- REF**, REF**1, REF**10, REF**11, REF**12, REF**13, REF**14, REF**15, REF**16, REF**17, REF**18, REF**19, REF**2, REF**20, REF**21, REF**22, REF**23, REF**24, REF**25, REF**26, REF**27, REF**28, REF**29, REF**3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: footprint Library:Switch_Hole -> Library:Switch_Hole5
- moved REF** 50.8 mm to (79.4, 41.3)
Routing:
- added copper zone on B.Cu, net (none)
- added copper zone on F.Cu, net (none)
