File: PCB/V4/34/34.kicad_pcb (KiCad board)
At the start: 2 copper layers, 112.4 x 93.3 mm, 61 parts, among them J1 USB_C_Receptacle_USB2.0, J2 Conn_01x04, J3 AVR-ISP-6, J4 Conn_01x04, SW1 SW_Push, SW10 SW_Push, SW11 SW_Push, SW12 SW_Push, SW13 SW_Push, SW14 SW_Push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

Commit message: right hand ready
Parts:
- moved J4 0.41 mm to (243.8, 45.6)
- moved C4 0.20 mm to (217.5, 128.2)
Connections:
- U1 pad 25: unconnected-(U1-Pad25) -> Row4
- U1 pad 26: unconnected-(U1-Pad26) -> Col6
- U1 pad 27: unconnected-(U1-Pad27) -> Col7
- U1 pad 36: unconnected-(U1-Pad36) -> Row1
- U1 pad 37: unconnected-(U1-Pad37) -> Row2
- U1 pad 38: unconnected-(U1-Pad38) -> Row3
- U1 pad 39: unconnected-(U1-Pad39) -> Col8
- U1 pad 40: unconnected-(U1-Pad40) -> Col9
- U1 pad 41: unconnected-(U1-Pad41) -> Col10
Routing:
- net Col6: track 0.00 -> 124.1 mm, vias 0 -> 5
- net Row1: track 22.4 -> 142.6 mm, vias 0 -> 4
- net Col7: track 0.00 -> 100.8 mm, vias 0 -> 2
- net Row2: track 22.9 -> 122.4 mm, vias 0 -> 2
- net Row3: track 0.00 -> 99.1 mm
- net Col8: track 0.00 -> 75.6 mm, vias 0 -> 3
- net Row4: track 0.00 -> 44.1 mm, vias 0 -> 2
- net Col10: track 67.8 -> 110.8 mm, vias 0 -> 3
- net Col9: track 50.2 -> 83.5 mm, vias 0 -> 3
- net Net-(D13-Pad2): track 0.00 -> 16.4 mm
- net Net-(D6-Pad2): track 0.00 -> 16.4 mm
- net Net-(D8-Pad2): track 0.00 -> 16.4 mm
- net Net-(D7-Pad2): track 0.00 -> 16.4 mm
- net Net-(D14-Pad2): track 0.00 -> 16.4 mm
- net Net-(D5-Pad2): track 0.00 -> 16.4 mm
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