File: PCB/V3/Input 34 Left plate/Pragmatic.kicad_pcb (KiCad board)
At the start: 2 copper layers, 109.9 x 90.8 mm, 22 parts, among them SW1 SW_Push, SW10 SW_Push, SW11 SW_Push, SW13 SW_Push, SW14 SW_Push, SW15 SW_Push, SW16 SW_Push, SW17 SW_Push, SW2 SW_Push, SW22 SW_Push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

Commit message: v3.1 34
Parts:
- SW1, SW10, SW11, SW13, SW14, SW15, SW16, SW17, SW2, SW22, SW23, SW3, SW4, SW5, SW7, SW8, SW9: footprint Pragmatic:Switch_Hole_Cutout_w_Deco -> Keyboard_JSA:Switch_Hole_Cutout_w_Deco
- moved H4 4.44 mm to (128.9, 114.3)
- moved H1 0.89 mm to (67.6, 76.2)
- moved H2 0.89 mm to (65.8, 104.8)
Other:
- board text added: "https://github.com/ jamessa/Pragmatic"
- board text removed: "Ergo input by James Sa https://github.com/ jamessa/Pragmatic"
