File: PCB/V3/Input 6x6/Pragmatic.kicad_sch (KiCad schematic)
At the start: 80 parts, among them J1 Hand-Soldering, SW1 SW_Push, SW10 SW_Push, SW11 SW_Push, SW12 SW_Push, SW13 SW_Push, SW14 SW_Push, SW15 SW_Push, SW16 SW_Push, SW17 SW_Push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

Commit message: increase plate border for manufacture.
Parts:
- SW1, SW10, SW11, SW12, SW13, SW14, SW15, SW16, SW17, SW18, SW19, SW2, SW20, SW21, SW22, SW23, SW24, SW25, SW26, SW27, SW28, SW29, SW3, SW30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: footprint (none) -> Keyboard_JSA:MX_Hotswap_MX_Choc_Solder
