File: PCB/V3/Control with OLED/Control.kicad_sch (KiCad schematic)
At the start: 6 parts, among them J1 L, J2 R, J3 OLED, J4 OLED, SW1 SW_Push, U1 ProMicro

Commit message: update border.
Parts:
- U1: footprint Keyboard_JSA:ProMicro Reversed -> Keyboard_JSA:ProMicro Type C Reversed
Changed lines of the file:
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@@
       (effects (font (size 1.524 1.524)))
     )
-    (property "Footprint" "Keyboard_JSA:ProMicro Reversed" (id 2) (at 166.37 161.29 90)
+    (property "Footprint" "Keyboard_JSA:ProMicro Type C Reversed" (id 2) (at 166.37 161.29 90)
       (effects (font (size 1.524 1.524)) hide)
     )
@@
     )
     (path "/c77559f1-9310-438e-bb42-9cac3de0d116"
-      (reference "U1") (unit 1) (value "ProMicro") (footprint "Keyboard_JSA:ProMicro Reversed")
+      (reference "U1") (unit 1) (value "ProMicro") (footprint "Keyboard_JSA:ProMicro Type C Reversed")
     )
   )
