File: PCB/V3/Input 34a left plate/Pragmatic.kicad_pcb (KiCad board)
At the start: 2 copper layers, 109.9 x 100.3 mm, 22 parts, among them SW1 SW_Push, SW10 SW_Push, SW11 SW_Push, SW13 SW_Push, SW14 SW_Push, SW15 SW_Push, SW16 SW_Push, SW17 SW_Push, SW2 SW_Push, SW22 SW_Push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

Commit message: almost there
Parts:
- moved H4 10.5 mm to (133.3, 123.8)
- moved LOGO1 5.72 mm to (95.2, 114.3)
Other:
- outline, holes or cut-outs redrawn
- board text removed: "https://github.com/ jamessa/Pragmatic"
Changed lines of the file:
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@@
   )
   (footprint "MountingHole:MountingHole_2.5mm" (layer "F.Cu")
-    (at 128.905 114.3)
+    (at 133.35 123.825)
     (descr "Mounting Hole 2.5mm, no annular")
     (tags "mounting hole 2.5mm no annular")
@@
       (effects (font (size 1 1) (thickness 0.15)))
     )
-    (fp_text value "MountingHole" (at 0 3.5) (layer "F.Fab")
+    (fp_text value "MountingHole" (at 0 3.5) (layer "F.Fab") hide
       (effects (font (size 1 1) (thickness 0.15)))
     )
-    (fp_text user "${REFERENCE}" (at 0.3 0) (layer "F.Fab")
+    (fp_text user "${REFERENCE}" (at 0.3 0) (layer "F.Fab") hide
       (effects (font (size 1 1) (thickness 0.15)))
     )
@@
   )
   (footprint "Symbol:OSHW-Logo_5.7x6mm_Copper" (layer "F.Cu")
-    (at 95.25 108.585)
+    (at 95.25 114.3)
     (descr "Open Source Hardware Logo")
     (tags "Logo OSHW")
@@
       ) (layer "F.Mask") (width 0.01) (fill solid))
   )
-  (gr_line (start 66.675 54.61) (end 80.645 54.61) (layer "Edge.Cuts") (width 0.12))
+  (gr_rect (start 83.185 42.545) (end 88.265 47.625) (layer "Cmts.User") (width 0.12) (fill none))
+  (gr_rect (start 42.545 64.135) (end 47.625 69.215) (layer "Cmts.User") (width 0.12) (fill none))
+  (gr_rect (start 92.71 123.825) (end 97.79 128.905) (layer "Cmts.User") (width 0.12) (fill none))
+  (gr_rect (start 152.4 142.875) (end 157.48 147.955) (layer "Cmts.User") (width 0.12) (fill none))
+  (gr_rect (start 142.875 111.76) (end 147.955 116.84) (layer "Cmts.User") (width 0.12) (fill none))
+  (gr_rect (start 152.4 121.285) (end 157.48 126.365) (layer "Cmts.User") (width 0.12) (fill none))
+  (gr_rect (start 111.76 142.875) (end 116.84 147.955) (layer "Cmts.User") (width 0.12) (fill none))
   (gr_line (start 107.315 52.07) (end 107.315 47.625) (layer "Edge.Cuts") (width 0.12))
-  (gr_line (start 45.085 66.675) (end 45.085 142.875) (layer "Edge.Cuts") (width 0.12))
-  (gr_arc (start 147.955 111.76) (mid 146.158949 111.016051) (end 145.415 109.22) (layer "Edge.Cuts") (width 0.12))
+  (gr_line (start 45.085 69.215) (end 45.085 123.825) (layer "Edge.Cuts") (width 0.12))
   (gr_arc (start 109.855 54.61) (mid 108.058949 53.866051) (end 107.315 52.07) (layer "Edge.Cuts") (width 0.12))
-  (gr_arc (start 152.4 111.76) (mid 154.196051 112.503949) (end 154.94 114.3) (layer "Edge.Cuts") (width 0.12))
-  (gr_line (start 152.4 111.76) (end 147.955 111.76) (layer "Edge.Cuts") (width 0.12))
-  (gr_line (start 83.185 52.07) (end 83.185 47.625) (layer "Edge.Cuts") (width 0.12))
-  (gr_line (start 64.135 57.15) (end 64.135 61.595) (layer "Edge.Cuts") (width 0.12))
-  (gr_arc (start 45.085 66.675) (mid 45.828949 64.878949) (end 47.625 64.135) (layer "Edge.Cuts") (width 0.12))
+  (gr_arc (start 116.84 145.414999) (mid 114.062765 144.619469) (end 111.760001 142.875) (layer "Edge.Cuts") (width 0.12))
+  (gr_line (start 152.4 121.285) (end 147.955 116.84) (layer "Edge.Cuts") (width 0.12))
   (gr_arc (start 104.775 45.085) (mid 106.571051 45.828949) (end 107.315 47.625) (layer "Edge.Cuts") (width 0.12))
-  (gr_arc (start 47.625 145.415) (mid 45.828949 144.671051) (end 45.085 142.875) (layer "Edge.Cuts") (width 0.12))
+  (gr_arc (start 47.625 126.365) (mid 45.828949 125.621051) (end 45.085 123.825) (layer "Edge.Cuts") (width 0.12))
+  (gr_line (start 83.185 46.355) (end 47.625 65.405) (layer "Edge.Cuts") (width 0.12))
   (gr_arc (start 142.875 54.61) (mid 144.671051 55.353949) (end 145.415 57.15) (layer "Edge.Cuts") (width 0.12))
-  (gr_arc (start 64.135 61.595) (mid 63.391051 63.391051) (end 61.595 64.135) (layer "Edge.Cuts") (width 0.12))
+  (gr_arc (start 147.955 116.839999) (mid 146.160183 114.562404) (end 145.415 111.76) (layer "Edge.Cuts") (width 0.12))
   (gr_line (start 109.855 54.61) (end 142.875 54.61) (layer "Edge.Cuts") (width 0.12))
-  (gr_line (start 154.94 116.84) (end 154.94 114.3) (layer "Edge.Cuts") (width 0.12))
+  (gr_arc (start 152.4 121.285) (mid 154.27985 123.520075) (end 154.94 126.365) (layer "Edge.Cuts") (width 0.12))
+  (gr_line (start 92.71 126.365) (end 47.625 126.365) (layer "Edge.Cuts") (width 0.12))
+  (gr_arc (start 92.71 126.365) (mid 95.459957 127.215087) (end 97.79 128.905) (layer "Edge.Cuts") (width 0.12))
+  (gr_arc (start 83.185 46.355) (mid 85.654113 45.436449) (end 88.265 45.085) (layer "Edge.Cuts") (width 0.12))
   (gr_arc (start 154.94 142.875) (mid 154.196051 144.671051) (end 152.4 145.415) (layer "Edge.Cuts") (width 0.12))
-  (gr_line (start 154.94 116.84) (end 154.94 142.875) (layer "Edge.Cuts") (width 0.12))
-  (gr_line (start 104.775 45.085) (end 85.725 45.085) (layer "Edge.Cuts") (width 0.12))
-  (gr_line (start 152.4 145.415) (end 47.625 145.415) (layer "Edge.Cuts") (width 0.12))
-  (gr_arc (start 64.135 57.15) (mid 64.878949 55.353949) (end 66.675 54.61) (layer "Edge.Cuts") (width 0.12))
-  (gr_arc (start 83.185 47.625) (mid 83.928949 45.828949) (end 85.725 45.085) (layer "Edge.Cuts") (width 0.12))
-  (gr_line (start 61.595 64.135) (end 47.625 64.135) (layer "Edge.Cuts") (width 0.12))
-  (gr_line (start 145.415 109.22) (end 145.415 57.15) (layer "Edge.Cuts") (width 0.12))
-  (gr_arc (start 83.185 52.07) (mid 82.441051 53.866051) (end 80.645 54.61) (layer "Edge.Cuts") (width 0.12))
-  (gr_text "https://github.com/\njamessa/Pragmatic" (at 95.25 108.585) (layer "B.SilkS")
-    (effects (font (size 1 1) (thickness 0.15)) (justify mirror))
-  )
+  (gr_line (start 154.94 126.365) (end 154.94 142.875) (layer "Edge.Cuts") (width 0.12))
+  (gr_line (start 104.775 45.085) (end 88.265 45.085) (layer "Edge.Cuts") (width 0.12))
+  (gr_line (start 152.4 145.415) (end 116.84 145.415) (layer "Edge.Cuts") (width 0.12))
+  (gr_line (start 97.79 128.905) (end 111.76 142.875) (layer "Edge.Cuts") (width 0.12))
+  (gr_arc (start 45.085 69.215) (mid 45.778212 66.925475) (end 47.625 65.405) (layer "Edge.Cuts") (width 0.12))
+  (gr_line (start 145.415 111.76) (end 145.415 57.15) (layer "Edge.Cuts") (width 0.12))
   (gr_text "김" (at 68.58 93.98) (layer "B.SilkS")
     (effects (font (size 1 1) (thickness 0.15)) (justify mirror))
