File: PCB/V3/Input 34a/34a.kicad_pcb (KiCad board)
At the start: 2 copper layers, 222.2 x 110.5 mm, 84 parts, among them J1 Hand-Soldering, J2 Hand-Soldering, SW1 SW_Push, SW10 SW_Push, SW11 SW_Push, SW12 SW_Push, SW13 SW_Push, SW14 SW_Push, SW15 SW_Push, SW16 SW_Push, SW17 SW_Push, SW18 SW_Push, SW19 SW_Push, SW2 SW_Push, SW20 SW_Push, SW21 SW_Push, SW22 SW_Push, SW23 SW_Push, SW24 SW_Push, SW25 SW_Push, SW26 SW_Push, SW27 SW_Push, SW28 SW_Push, SW29 SW_Push, SW3 SW_Push, SW30 SW_Push, SW31 SW_Push, SW32 SW_Push, SW33 SW_Push, SW34 SW_Push, SW37 SW_Push, SW38 SW_Push, SW4 SW_Push, SW5 SW_Push, SW6 SW_Push, SW7 SW_Push, SW8 SW_Push, SW9 SW_Push

Commit message: ready for print
Parts:
- moved REF** 70.9 mm to (188.6, 119.8)
- moved LOGO1 70.4 mm to (123.8, 118.7)
Routing:
- net Row5': track 0.00 -> 161.2 mm, vias 0 -> 1
- net Row6: track 0.00 -> 159.2 mm, vias 0 -> 1
- net Row5: track 0.00 -> 158.9 mm, vias 0 -> 1
- net Row6': track 0.00 -> 143.5 mm, vias 0 -> 1
- net Row4: track 0.00 -> 142.8 mm, vias 0 -> 1
- net Row4': track 0.00 -> 139.5 mm, vias 0 -> 1
- net Col11: track 0.00 -> 123.9 mm
- net Row3: track 0.00 -> 122.9 mm, vias 0 -> 1
- net Col2: track 0.00 -> 113.6 mm, vias 0 -> 3
- net Row3': track 0.00 -> 113.0 mm, vias 0 -> 1
- net Col8: track 0.00 -> 108.4 mm, vias 0 -> 4
- net Col9: track 0.00 -> 106.0 mm, vias 0 -> 4
- net Col10: track 0.00 -> 105.3 mm, vias 0 -> 3
- net Col7: track 0.00 -> 95.9 mm, vias 0 -> 4
- net Col5: track 0.00 -> 93.0 mm, vias 0 -> 4
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Other:
- board text added: "Pragmatic 34a by James Sa"
