File: PCB/V3/Input 34a/34a.kicad_sch (KiCad schematic)
At the start: 84 parts, among them J1 Hand-Soldering, J2 Hand-Soldering, SW1 SW_Push, SW10 SW_Push, SW11 SW_Push, SW12 SW_Push, SW13 SW_Push, SW14 SW_Push, SW15 SW_Push, SW16 SW_Push, SW17 SW_Push, SW18 SW_Push, SW19 SW_Push, SW2 SW_Push, SW20 SW_Push, SW21 SW_Push, SW22 SW_Push, SW23 SW_Push, SW24 SW_Push, SW25 SW_Push, SW26 SW_Push, SW27 SW_Push, SW28 SW_Push, SW29 SW_Push, SW3 SW_Push, SW30 SW_Push, SW31 SW_Push, SW32 SW_Push, SW33 SW_Push, SW34 SW_Push, SW37 SW_Push, SW38 SW_Push, SW4 SW_Push, SW5 SW_Push, SW6 SW_Push, SW7 SW_Push, SW8 SW_Push, SW9 SW_Push

Commit message: ready for print
Parts:
- removed H4, H7: MountingHole, MountingHole:MountingHole_2.5mm, symbol Mechanical:MountingHole
- renumbered H5 to H4, H6 to H5, H8 to H6, H9 to H7, H10 to H8
Other:
- moved on the sheet: H1, H2, H3, H4, H5
Changed lines of the file:
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@@
     (pin "9")
   )
-  (symbol (lib_id "Mechanical:MountingHole") (at 214.63 127 0) (unit 1)
-    (in_bom yes) (on_board yes)
-    (property "Reference" "H1" (id 0) (at 217.17 125.8316 0)
+  (symbol (lib_id "Mechanical:MountingHole") (at 215.9 133.35 0) (unit 1)
+    (in_bom yes) (on_board yes)
+    (property "Reference" "H1" (id 0) (at 218.44 132.1816 0)
       (effects (font (size 1.27 1.27)) (justify left))
     )
-    (property "Value" "MountingHole" (id 1) (at 217.17 128.143 0)
+    (property "Value" "MountingHole" (id 1) (at 218.44 134.493 0)
       (effects (font (size 1.27 1.27)) (justify left) hide)
     )
-    (property "Footprint" "MountingHole:MountingHole_2.5mm" (id 2) (at 214.63 127 0)
-      (effects (font (size 1.27 1.27)) hide)
-    )
-    (property "Datasheet" "~" (id 3) (at 214.63 127 0)
-      (effects (font (size 1.27 1.27)) hide)
-    )
-  )
-  (symbol (lib_id "Mechanical:MountingHole") (at 214.63 133.35 0) (unit 1)
-    (in_bom yes) (on_board yes)
-    (property "Reference" "H2" (id 0) (at 217.17 132.1816 0)
+    (property "Footprint" "MountingHole:MountingHole_2.5mm" (id 2) (at 215.9 133.35 0)
+      (effects (font (size 1.27 1.27)) hide)
+    )
+    (property "Datasheet" "~" (id 3) (at 215.9 133.35 0)
+      (effects (font (size 1.27 1.27)) hide)
+    )
+  )
+  (symbol (lib_id "Mechanical:MountingHole") (at 215.9 139.7 0) (unit 1)
+    (in_bom yes) (on_board yes)
+    (property "Reference" "H2" (id 0) (at 218.44 138.5316 0)
       (effects (font (size 1.27 1.27)) (justify left))
     )
-    (property "Value" "MountingHole" (id 1) (at 217.17 134.493 0)
+    (property "Value" "MountingHole" (id 1) (at 218.44 140.843 0)
       (effects (font (size 1.27 1.27)) (justify left) hide)
     )
-    (property "Footprint" "MountingHole:MountingHole_2.5mm" (id 2) (at 214.63 133.35 0)
-      (effects (font (size 1.27 1.27)) hide)
-    )
-    (property "Datasheet" "~" (id 3) (at 214.63 133.35 0)
-      (effects (font (size 1.27 1.27)) hide)
-    )
-  )
-  (symbol (lib_id "Mechanical:MountingHole") (at 214.63 139.7 0) (unit 1)
-    (in_bom yes) (on_board yes)
-    (property "Reference" "H3" (id 0) (at 217.17 138.5316 0)
+    (property "Footprint" "MountingHole:MountingHole_2.5mm" (id 2) (at 215.9 139.7 0)
+      (effects (font (size 1.27 1.27)) hide)
+    )
+    (property "Datasheet" "~" (id 3) (at 215.9 139.7 0)
+      (effects (font (size 1.27 1.27)) hide)
+    )
+  )
+  (symbol (lib_id "Mechanical:MountingHole") (at 215.9 146.05 0) (unit 1)
+    (in_bom yes) (on_board yes)
+    (property "Reference" "H3" (id 0) (at 218.44 144.8816 0)
       (effects (font (size 1.27 1.27)) (justify left))
     )
-    (property "Value" "MountingHole" (id 1) (at 217.17 140.843 0)
+    (property "Value" "MountingHole" (id 1) (at 218.44 147.193 0)
       (effects (font (size 1.27 1.27)) (justify left) hide)
     )
-    (property "Footprint" "MountingHole:MountingHole_2.5mm" (id 2) (at 214.63 139.7 0)
-      (effects (font (size 1.27 1.27)) hide)
-    )
-    (property "Datasheet" "~" (id 3) (at 214.63 139.7 0)
-      (effects (font (size 1.27 1.27)) hide)
-    )
-  )
-  (symbol (lib_id "Mechanical:MountingHole") (at 214.63 146.685 0) (unit 1)
-    (in_bom yes) (on_board yes)
-    (property "Reference" "H4" (id 0) (at 217.17 145.5166 0)
-      (effects (font (size 1.27 1.27)) (justify left))
-    )
-    (property "Value" "MountingHole" (id 1) (at 217.17 147.828 0)
-      (effects (font (size 1.27 1.27)) (justify left) hide)
-    )
-    (property "Footprint" "MountingHole:MountingHole_2.5mm" (id 2) (at 214.63 146.685 0)
-      (effects (font (size 1.27 1.27)) hide)
-    )
-    (property "Datasheet" "~" (id 3) (at 214.63 146.685 0)
+    (property "Footprint" "MountingHole:MountingHole_2.5mm" (id 2) (at 215.9 146.05 0)
+      (effects (font (size 1.27 1.27)) hide)
+    )
+    (property "Datasheet" "~" (id 3) (at 215.9 146.05 0)
       (effects (font (size 1.27 1.27)) hide)
     )
@@
     (pin "2")
   )
-  (symbol (lib_id "Mechanical:MountingHole") (at 214.63 152.4 0) (unit 1)
-    (in_bom yes) (on_board yes)
-    (property "Reference" "H5" (id 0) (at 217.17 151.2316 0)
+  (symbol (lib_id "Mechanical:MountingHole") (at 215.9 152.4 0) (unit 1)
+    (in_bom yes) (on_board yes)
+    (property "Reference" "H4" (id 0) (at 218.44 151.2316 0)
       (effects (font (size 1.27 1.27)) (justify left))
     )
-    (property "Value" "MountingHole" (id 1) (at 217.17 153.543 0)
+    (property "Value" "MountingHole" (id 1) (at 218.44 153.543 0)
       (effects (font (size 1.27 1.27)) (justify left) hide)
     )
-    (property "Footprint" "MountingHole:MountingHole_2.5mm" (id 2) (at 214.63 152.4 0)
-      (effects (font (size 1.27 1.27)) hide)
-    )
-    (property "Datasheet" "~" (id 3) (at 214.63 152.4 0)
+    (property "Footprint" "MountingHole:MountingHole_2.5mm" (id 2) (at 215.9 152.4 0)
+      (effects (font (size 1.27 1.27)) hide)
+    )
+    (property "Datasheet" "~" (id 3) (at 215.9 152.4 0)
       (effects (font (size 1.27 1.27)) hide)
     )
@@
   (symbol (lib_id "Mechanical:MountingHole") (at 226.06 139.7 0) (unit 1)
     (in_bom yes) (on_board yes)
-    (property "Reference" "H8" (id 0) (at 228.6 138.5316 0)
+    (property "Reference" "H6" (id 0) (at 228.6 138.5316 0)
       (effects (font (size 1.27 1.27)) (justify left))
     )
@@
     (pin "2")
   )
-  (symbol (lib_id "Mechanical:MountingHole") (at 226.06 127 0) (unit 1)
-    (in_bom yes) (on_board yes)
-    (property "Reference" "H6" (id 0) (at 228.6 125.8316 0)
+  (symbol (lib_id "Mechanical:MountingHole") (at 227.33 133.35 0) (unit 1)
+    (in_bom yes) (on_board yes)
+    (property "Reference" "H5" (id 0) (at 229.87 132.1816 0)
       (effects (font (size 1.27 1.27)) (justify left))
     )
-    (property "Value" "MountingHole" (id 1) (at 228.6 128.143 0)
+    (property "Value" "MountingHole" (id 1) (at 229.87 134.493 0)
       (effects (font (size 1.27 1.27)) (justify left) hide)
     )
-    (property "Footprint" "MountingHole:MountingHole_2.5mm" (id 2) (at 226.06 127 0)
-      (effects (font (size 1.27 1.27)) hide)
-    )
-    (property "Datasheet" "~" (id 3) (at 226.06 127 0)
-      (effects (font (size 1.27 1.27)) hide)
-    )
-  )
-  (symbol (lib_id "Mechanical:MountingHole") (at 226.06 133.35 0) (unit 1)
-    (in_bom yes) (on_board yes)
-    (property "Reference" "H7" (id 0) (at 228.6 132.1816 0)
-      (effects (font (size 1.27 1.27)) (justify left))
-    )
-    (property "Value" "MountingHole" (id 1) (at 228.6 134.493 0)
-      (effects (font (size 1.27 1.27)) (justify left) hide)
-    )
-    (property "Footprint" "MountingHole:MountingHole_2.5mm" (id 2) (at 226.06 133.35 0)
-      (effects (font (size 1.27 1.27)) hide)
-    )
-    (property "Datasheet" "~" (id 3) (at 226.06 133.35 0)
+    (property "Footprint" "MountingHole:MountingHole_2.5mm" (id 2) (at 227.33 133.35 0)
+      (effects (font (size 1.27 1.27)) hide)
+    )
+    (property "Datasheet" "~" (id 3) (at 227.33 133.35 0)
       (effects (font (size 1.27 1.27)) hide)
     )
@@
   (symbol (lib_id "Mechanical:MountingHole") (at 226.06 146.05 0) (unit 1)
     (in_bom yes) (on_board yes)
-    (property "Reference" "H9" (id 0) (at 228.6 144.8816 0)
+    (property "Reference" "H7" (id 0) (at 228.6 144.8816 0)
       (effects (font (size 1.27 1.27)) (justify left))
     )
@@
   (symbol (lib_id "Mechanical:MountingHole") (at 226.06 152.4 0) (unit 1)
     (in_bom yes) (on_board yes)
-    (property "Reference" "H10" (id 0) (at 228.6 151.2316 0)
+    (property "Reference" "H8" (id 0) (at 228.6 151.2316 0)
       (effects (font (size 1.27 1.27)) (justify left))
     )
@@
       (reference "H3") (unit 1) (value "MountingHole") (footprint "MountingHole:MountingHole_2.5mm")
     )
-    (path "/00000000-0000-0000-0000-000061be2ba9"
+    (path "/2cfc0c5a-9a31-4eba-adaa-31a9735947a9"
       (reference "H4") (unit 1) (value "MountingHole") (footprint "MountingHole:MountingHole_2.5mm")
     )
-    (path "/2cfc0c5a-9a31-4eba-adaa-31a9735947a9"
+    (path "/a26e4c66-9cc9-474e-8435-cc0650675de6"
       (reference "H5") (unit 1) (value "MountingHole") (footprint "MountingHole:MountingHole_2.5mm")
     )
-    (path "/a26e4c66-9cc9-474e-8435-cc0650675de6"
+    (path "/6c468d70-5bc7-46e3-94ff-14dc764c3d8d"
       (reference "H6") (unit 1) (value "MountingHole") (footprint "MountingHole:MountingHole_2.5mm")
     )
-    (path "/a57bdcc1-7a14-44e2-bb52-e2c0ae0ec1af"
+    (path "/b7cd54c4-314f-4c5a-bf1e-ba3b7a7ce2bb"
       (reference "H7") (unit 1) (value "MountingHole") (footprint "MountingHole:MountingHole_2.5mm")
     )
-    (path "/6c468d70-5bc7-46e3-94ff-14dc764c3d8d"
+    (path "/ca91c247-dc80-4a25-befb-9245548cce18"
       (reference "H8") (unit 1) (value "MountingHole") (footprint "MountingHole:MountingHole_2.5mm")
     )
-    (path "/b7cd54c4-314f-4c5a-bf1e-ba3b7a7ce2bb"
-      (reference "H9") (unit 1) (value "MountingHole") (footprint "MountingHole:MountingHole_2.5mm")
-    )
-    (path "/ca91c247-dc80-4a25-befb-9245548cce18"
-      (reference "H10") (unit 1) (value "MountingHole") (footprint "MountingHole:MountingHole_2.5mm")
-    )
     (path "/00000000-0000-0000-0000-000061aaace1"
