File: PCB/V3/Input 34a plate left/Plate.kicad_pcb (KiCad board)
At the start: 2 copper layers, 109.9 x 100.3 mm, 22 parts, among them SW1 SW_Push, SW10 SW_Push, SW11 SW_Push, SW13 SW_Push, SW14 SW_Push, SW15 SW_Push, SW16 SW_Push, SW17 SW_Push, SW2 SW_Push, SW22 SW_Push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

Commit message: update logo
Parts:
- moved REF** 1.27 mm to (95.2, 119.4)
