File: Pragmatic34/Input 34a/34a.kicad_pcb (KiCad board)
At the start: 2 copper layers, 222.2 x 110.5 mm, 84 parts, among them J1 Hand-Soldering, J2 Hand-Soldering, SW1 SW_Push, SW10 SW_Push, SW11 SW_Push, SW12 SW_Push, SW13 SW_Push, SW14 SW_Push, SW15 SW_Push, SW16 SW_Push, SW17 SW_Push, SW18 SW_Push, SW19 SW_Push, SW2 SW_Push, SW20 SW_Push, SW21 SW_Push, SW22 SW_Push, SW23 SW_Push, SW24 SW_Push, SW25 SW_Push, SW26 SW_Push, SW27 SW_Push, SW28 SW_Push, SW29 SW_Push, SW3 SW_Push, SW30 SW_Push, SW31 SW_Push, SW32 SW_Push, SW33 SW_Push, SW34 SW_Push, SW37 SW_Push, SW38 SW_Push, SW4 SW_Push, SW5 SW_Push, SW6 SW_Push, SW7 SW_Push, SW8 SW_Push, SW9 SW_Push

Commit message: simplify
Parts:
- removed D37, D38: 1N4148, Keyboard_Foostan:D3_SMD_v2
- removed SW37, SW38: SW_Push, Keyboard_JSA:MX_Hotswap
- added REF**: Fiducial_1mm_Mask2mm, Fiducial:Fiducial_1mm_Mask2mm, B.Cu at (262.9, 43.8)
- added REF**: Fiducial_1mm_Mask2mm, Fiducial:Fiducial_1mm_Mask2mm, B.Cu at (262.9, 146.7)
- added REF**: Fiducial_1mm_Mask2mm, Fiducial:Fiducial_1mm_Mask2mm, B.Cu at (49.5, 43.8)
- added REF**: Fiducial_1mm_Mask2mm, Fiducial:Fiducial_1mm_Mask2mm, B.Cu at (49.5, 146.7)
Routing:
- net VCC: track 83.1 -> 0.00 mm
- net GND: track 69.6 -> 0.00 mm
- net Row6: track 159.2 -> 120.6 mm
- net Col9: track 106.0 -> 84.5 mm, vias 4 -> 3
- net Col4: track 90.8 -> 70.0 mm, vias 4 -> 3
- net Row6': track 143.5 -> 127.9 mm
- net Net-(D38-Pad2): track 11.7 -> 0.00 mm
- net Net-(D37-Pad2): track 11.7 -> 0.00 mm
Other:
- board text added: "Pragmatic 34"
- board text added: "Revision 2"
- board text removed: "Pragmatic 34a by James Sa"
- board text removed: "V3.2"
