File: Pragmatic34/Input 34a/34a.kicad_sch (KiCad schematic)
At the start: 82 parts, among them J1 Hand-Soldering, J2 Hand-Soldering, SW1 SW_Push, SW10 SW_Push, SW11 SW_Push, SW12 SW_Push, SW13 SW_Push, SW14 SW_Push, SW15 SW_Push, SW16 SW_Push, SW17 SW_Push, SW18 SW_Push, SW19 SW_Push, SW2 SW_Push, SW20 SW_Push, SW21 SW_Push, SW22 SW_Push, SW23 SW_Push, SW24 SW_Push, SW25 SW_Push, SW26 SW_Push, SW27 SW_Push, SW28 SW_Push, SW29 SW_Push, SW3 SW_Push, SW30 SW_Push, SW31 SW_Push, SW32 SW_Push, SW33 SW_Push, SW34 SW_Push, SW37 SW_Push, SW38 SW_Push, SW4 SW_Push, SW5 SW_Push, SW6 SW_Push, SW7 SW_Push, SW8 SW_Push, SW9 SW_Push

Commit message: simplify
Parts:
- removed D37, D38: 1N4148, Keyboard_Foostan:D3_SMD_v2, symbol Device:D
- removed SW37, SW38: SW_Push, Keyboard_JSA:MX_Hotswap, symbol Switch:SW_Push
Changed lines of the file:
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@@
   (junction (at 73.66 76.2) (diameter 0) (color 0 0 0 0)
   )
-  (junction (at 148.59 129.54) (diameter 0) (color 0 0 0 0)
-  )
   (junction (at 76.2 99.06) (diameter 0) (color 0 0 0 0)
   )
@@
   (junction (at 60.96 76.2) (diameter 0) (color 0 0 0 0)
   )
-  (junction (at 171.45 106.68) (diameter 0) (color 0 0 0 0)
-  )
   (junction (at 99.06 76.2) (diameter 0) (color 0 0 0 0)
   )
@@
   (junction (at 60.96 91.44) (diameter 0) (color 0 0 0 0)
   )
-  (junction (at 86.36 106.68) (diameter 0) (color 0 0 0 0)
-  )
   (junction (at 111.76 91.44) (diameter 0) (color 0 0 0 0)
   )
   (junction (at 173.99 99.06) (diameter 0) (color 0 0 0 0)
-  )
-  (junction (at 76.2 129.54) (diameter 0) (color 0 0 0 0)
   )
   (junction (at 86.36 76.2) (diameter 0) (color 0 0 0 0)
@@
     (stroke (width 0) (type default) (color 0 0 0 0))
   )
-  (wire (pts (xy 76.2 129.54) (xy 88.9 129.54))
+  (wire (pts (xy 43.18 129.54) (xy 88.9 129.54))
     (stroke (width 0) (type default) (color 0 0 0 0))
   )
@@
     (stroke (width 0) (type default) (color 0 0 0 0))
   )
-  (wire (pts (xy 171.45 106.68) (xy 171.45 121.92))
-    (stroke (width 0) (type default) (color 0 0 0 0))
-  )
   (wire (pts (xy 99.06 91.44) (xy 99.06 106.68))
     (stroke (width 0) (type default) (color 0 0 0 0))
@@
     (stroke (width 0) (type default) (color 0 0 0 0))
   )
-  (wire (pts (xy 148.59 129.54) (xy 161.29 129.54))
-    (stroke (width 0) (type default) (color 0 0 0 0))
-  )
   (wire (pts (xy 76.2 99.06) (xy 88.9 99.06))
     (stroke (width 0) (type default) (color 0 0 0 0))
@@
     (stroke (width 0) (type default) (color 0 0 0 0))
   )
-  (wire (pts (xy 86.36 106.68) (xy 86.36 121.92))
-    (stroke (width 0) (type default) (color 0 0 0 0))
-  )
   (wire (pts (xy 171.45 91.44) (xy 171.45 106.68))
     (stroke (width 0) (type default) (color 0 0 0 0))
@@
   )
   (wire (pts (xy 130.81 114.3) (xy 135.89 114.3))
-    (stroke (width 0) (type default) (color 0 0 0 0))
-  )
-  (wire (pts (xy 43.18 129.54) (xy 76.2 129.54))
     (stroke (width 0) (type default) (color 0 0 0 0))
   )
@@
     )
   )
-  (symbol (lib_id "Device:D") (at 76.2 125.73 90) (unit 1)
-    (in_bom yes) (on_board yes)
-    (property "Reference" "D37" (id 0) (at 78.232 125.73 90)
-      (effects (font (size 1.27 1.27)) (justify right))
-    )
-    (property "Value" "1N4148" (id 1) (at 72.9996 125.73 0)
-      (effects (font (size 1.27 1.27)) hide)
-    )
-    (property "Footprint" "Keyboard_Foostan:D3_SMD_v2" (id 2) (at 76.2 125.73 0)
-      (effects (font (size 1.27 1.27)) hide)
-    )
-    (property "Datasheet" "~" (id 3) (at 76.2 125.73 0)
-      (effects (font (size 1.27 1.27)) hide)
-    )
-    (property "LCSC" "C81598" (id 4) (at 76.2 125.73 0)
-      (effects (font (size 1.27 1.27)) hide)
-    )
-    (pin "1")
-    (pin "2")
-  )
   (symbol (lib_id "Switch:SW_Push") (at 153.67 91.44 0) (unit 1)
     (in_bom yes) (on_board yes)
@@
       (effects (font (size 1.27 1.27)) hide)
     )
-  )
-  (symbol (lib_id "Switch:SW_Push") (at 166.37 121.92 0) (unit 1)
-    (in_bom yes) (on_board yes)
-    (property "Reference" "SW38" (id 0) (at 166.37 117.0178 0))
-    (property "Value" "SW_Push" (id 1) (at 166.37 116.9924 0)
-      (effects (font (size 1.27 1.27)) hide)
-    )
-    (property "Footprint" "Keyboard_JSA:MX_Hotswap" (id 2) (at 166.37 116.84 0)
-      (effects (font (size 1.27 1.27)) hide)
-    )
-    (property "Datasheet" "~" (id 3) (at 166.37 116.84 0)
-      (effects (font (size 1.27 1.27)) hide)
-    )
-    (pin "1")
-    (pin "2")
   )
   (symbol (lib_id "Device:D") (at 173.99 80.01 90) (unit 1)
@@
     )
   )
-  (symbol (lib_id "Switch:SW_Push") (at 81.28 121.92 0) (unit 1)
-    (in_bom yes) (on_board yes)
-    (property "Reference" "SW37" (id 0) (at 81.28 117.0178 0))
-    (property "Value" "SW_Push" (id 1) (at 81.28 116.9924 0)
-      (effects (font (size 1.27 1.27)) hide)
-    )
-    (property "Footprint" "Keyboard_JSA:MX_Hotswap" (id 2) (at 81.28 116.84 0)
-      (effects (font (size 1.27 1.27)) hide)
-    )
-    (property "Datasheet" "~" (id 3) (at 81.28 116.84 0)
-      (effects (font (size 1.27 1.27)) hide)
-    )
-    (pin "1")
-    (pin "2")
-  )
   (symbol (lib_id "Device:D") (at 161.29 110.49 90) (unit 1)
     (in_bom yes) (on_board yes)
@@
     )
     (property "LCSC" "C81598" (id 4) (at 135.89 125.73 0)
-      (effects (font (size 1.27 1.27)) hide)
-    )
-    (pin "1")
-    (pin "2")
-  )
-  (symbol (lib_id "Device:D") (at 161.29 125.73 90) (unit 1)
-    (in_bom yes) (on_board yes)
-    (property "Reference" "D38" (id 0) (at 163.322 125.73 90)
-      (effects (font (size 1.27 1.27)) (justify right))
-    )
-    (property "Value" "1N4148" (id 1) (at 158.0896 125.73 0)
-      (effects (font (size 1.27 1.27)) hide)
-    )
-    (property "Footprint" "Keyboard_Foostan:D3_SMD_v2" (id 2) (at 161.29 125.73 0)
-      (effects (font (size 1.27 1.27)) hide)
-    )
-    (property "Datasheet" "~" (id 3) (at 161.29 125.73 0)
-      (effects (font (size 1.27 1.27)) hide)
-    )
-    (property "LCSC" "C81598" (id 4) (at 161.29 125.73 0)
       (effects (font (size 1.27 1.27)) hide)
     )
@@
       (reference "D34") (unit 1) (value "1N4148") (footprint "Keyboard_Foostan:D3_SMD_v2")
     )
-    (path "/05acc916-31ae-4ffc-ab80-9b7244877240"
-      (reference "D37") (unit 1) (value "1N4148") (footprint "Keyboard_Foostan:D3_SMD_v2")
-    )
-    (path "/ec140271-5f27-4456-a863-fb4343827158"
-      (reference "D38") (unit 1) (value "1N4148") (footprint "Keyboard_Foostan:D3_SMD_v2")
-    )
     (path "/00000000-0000-0000-0000-000061bdfa75"
       (reference "H1") (unit 1) (value "MountingHole") (footprint "MountingHole:MountingHole_2.5mm")
@@
       (reference "SW34") (unit 1) (value "SW_Push") (footprint "Keyboard_JSA:MX_Hotswap")
     )
-    (path "/c3d92f6e-0d59-4b76-8b3d-c5d89c201403"
-      (reference "SW37") (unit 1) (value "SW_Push") (footprint "Keyboard_JSA:MX_Hotswap")
-    )
-    (path "/408d002a-4b68-44a0-b4f2-903124b3efdb"
-      (reference "SW38") (unit 1) (value "SW_Push") (footprint "Keyboard_JSA:MX_Hotswap")
-    )
-  )
+  )
