File: Pragmatic34/Input/Input.kicad_pcb (KiCad board)
At the start: 2 copper layers, 222.2 x 110.5 mm, 84 parts, among them J1 Hand-Soldering, J2 Hand-Soldering, SW1 SW_Push, SW10 SW_Push, SW11 SW_Push, SW12 SW_Push, SW13 SW_Push, SW14 SW_Push, SW15 SW_Push, SW16 SW_Push, SW17 SW_Push, SW18 SW_Push, SW19 SW_Push, SW2 SW_Push, SW20 SW_Push, SW21 SW_Push, SW22 SW_Push, SW23 SW_Push, SW24 SW_Push, SW25 SW_Push, SW26 SW_Push, SW27 SW_Push, SW28 SW_Push, SW29 SW_Push, SW3 SW_Push, SW30 SW_Push, SW31 SW_Push, SW32 SW_Push, SW33 SW_Push, SW34 SW_Push, SW4 SW_Push, SW5 SW_Push, SW6 SW_Push, SW7 SW_Push, SW8 SW_Push, SW9 SW_Push

Commit message: fix rubber position
Parts:
- SW1, SW10, SW11, SW12, SW13, SW14, SW15, SW16, SW17, SW18, SW19, SW2, SW20, SW21, SW22, SW23, SW24, SW25, SW26, SW27, SW28, SW29, SW3, SW30, SW31, SW32, SW33, SW34, SW4, SW5, SW6, SW7, SW8, SW9: moved to B.Cu
- moved D10 14.6 mm to (255.3, 69.2)
- moved D1 14.1 mm to (57.1, 69.1)
- turned SW11 to 180 degrees
- turned SW12 to 180 degrees
- turned SW13 to 180 degrees
- turned SW14 to 180 degrees
- turned SW15 to 180 degrees
- turned SW16 to 180 degrees
- turned SW17 to 180 degrees
- turned SW18 to 180 degrees
- turned SW19 to 180 degrees
- turned SW2 to 180 degrees
- turned SW20 to 180 degrees
- turned SW21 to 180 degrees
- turned SW22 to 180 degrees
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Routing:
- net Col2: track 113.6 -> 110.9 mm, vias 3 -> 4
- net Net-(D1-Pad2): track 11.7 -> 13.9 mm
- net Row3': track 113.0 -> 111.0 mm
- net Row3: track 122.9 -> 121.3 mm
- net Net-(D10-Pad2): track 12.4 -> 13.7 mm
- net Col10: track 105.3 -> 106.3 mm
- net Col11: track 123.9 -> 123.3 mm
