File: Pragmatic34/Control with OLED/Control.kicad_pcb (KiCad board)
At the start: 2 copper layers, 41.9 x 48.3 mm, 9 parts, among them J1 L, J2 R, J3 OLED, J4 OLED, SW1 SW_Push, U1 ProMicro

Commit message: update control board
Parts:
- added REF**: logo, Keyboard_JSA:Pragmatic Logo, F.Cu at (139.9, 89.5)
- Logo1: value OSHW-Logo2_7.3x6mm_Copper -> OSHW-Symbol_6.7x6mm_Copper; footprint keyboards:OSHW-Logo2_7.3x6mm_Copper -> Symbol:OSHW-Symbol_6.7x6mm_Copper
- REF**: value KiCad-Logo_5mm_Copper -> KiCad-Logo_5mm_SilkScreen; footprint Symbol:KiCad-Logo_5mm_Copper -> Symbol:KiCad-Logo_5mm_SilkScreen
- turned REF** to 135 degrees
Other:
- board text removed: "Pragmatic"
