File: Anya/Anya.kicad_sch (KiCad schematic)
At the start: 76 parts, among them SW1 SW_Push, SW10 SW_Push, SW11 SW_Push, SW12 SW_Push, SW13 SW_Push, SW14 SW_Push, SW15 SW_Push, SW16 SW_Push, SW17 SW_Push, SW18 SW_Push, SW19 SW_Push, SW2 SW_Push, SW20 SW_Push, SW21 SW_Push, SW22 SW_Push, SW23 SW_Push, SW24 SW_Push, SW25 SW_Push, SW26 SW_Push, SW27 SW_Push, SW28 SW_Push, SW29 SW_Push, SW3 SW_Push, SW30 SW_Push, SW31 SW_Push, SW32 SW_Push, SW33 SW_Push, SW4 SW_Push, SW5 SW_Push, SW6 SW_Push, SW7 SW_Push, SW8 SW_Push, SW9 SW_Push, U1 ProMicro

Commit message: Anya R1
Connections:
- net Col 10: now also U1.13 (10/PB6); no longer U1.18 (A1/PF6)
- net Col 8: now also U1.15 (14/PB3); no longer U1.20 (A3/PF4)
- net Col 9: now also U1.14 (16/PB2); no longer U1.19 (A2/PF5)
- net Left: now also U1.17 (A0/PF7); no longer U1.13 (10/PB6)
- net Middle: now also U1.18 (A1/PF6); no longer U1.14 (16/PB2)
- net Right: now also U1.19 (A2/PF5); no longer U1.15 (14/PB3)
- net Row 4: now also U1.16 (15/PB1); no longer U1.17 (A0/PF7)
- no-connect marks 3 -> 2
Changed lines of the file:
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@@
   )
   (no_connect (at 73.66 119.38))
-  (no_connect (at 73.66 134.62))
   (no_connect (at 73.66 114.3))
   (wire (pts (xy 233.68 83.82) (xy 248.92 83.82))
@@
     )
   )
-  (global_label "Col 10" (shape input) (at 73.66 129.54 0) (fields_autoplaced)
-    (effects (font (size 1.27 1.27)) (justify left))
-    (property "Intersheetrefs" "${INTERSHEET_REFS}" (at 83.0366 129.54 0)
-      (effects (font (size 1.27 1.27)) (justify left) hide)
-    )
-  )
-  (global_label "Right" (shape input) (at 73.66 137.16 0) (fields_autoplaced)
-    (effects (font (size 1.27 1.27)) (justify left))
-    (property "Intersheetrefs" "${INTERSHEET_REFS}" (at 81.4643 137.16 0)
+  (global_label "Col 10" (shape input) (at 73.66 142.24 0) (fields_autoplaced)
+    (effects (font (size 1.27 1.27)) (justify left))
+    (property "Intersheetrefs" "${INTERSHEET_REFS}" (at 83.0366 142.24 0)
+      (effects (font (size 1.27 1.27)) (justify left) hide)
+    )
+  )
+  (global_label "Right" (shape input) (at 73.66 127 0) (fields_autoplaced)
+    (effects (font (size 1.27 1.27)) (justify left))
+    (property "Intersheetrefs" "${INTERSHEET_REFS}" (at 81.4643 127 0)
       (effects (font (size 1.27 1.27)) (justify left) hide)
     )
@@
     )
   )
-  (global_label "Middle" (shape input) (at 73.66 139.7 0) (fields_autoplaced)
-    (effects (font (size 1.27 1.27)) (justify left))
-    (property "Intersheetrefs" "${INTERSHEET_REFS}" (at 82.6738 139.7 0)
+  (global_label "Middle" (shape input) (at 73.66 129.54 0) (fields_autoplaced)
+    (effects (font (size 1.27 1.27)) (justify left))
+    (property "Intersheetrefs" "${INTERSHEET_REFS}" (at 82.6738 129.54 0)
       (effects (font (size 1.27 1.27)) (justify left) hide)
     )
@@
     )
   )
-  (global_label "Col 8" (shape input) (at 73.66 124.46 0) (fields_autoplaced)
-    (effects (font (size 1.27 1.27)) (justify left))
-    (property "Intersheetrefs" "${INTERSHEET_REFS}" (at 81.8271 124.46 0)
+  (global_label "Col 8" (shape input) (at 73.66 137.16 0) (fields_autoplaced)
+    (effects (font (size 1.27 1.27)) (justify left))
+    (property "Intersheetrefs" "${INTERSHEET_REFS}" (at 81.8271 137.16 0)
       (effects (font (size 1.27 1.27)) (justify left) hide)
     )
@@
     )
   )
-  (global_label "Row 4" (shape input) (at 73.66 132.08 0) (fields_autoplaced)
-    (effects (font (size 1.27 1.27)) (justify left))
-    (property "Intersheetrefs" "${INTERSHEET_REFS}" (at 82.4924 132.08 0)
+  (global_label "Row 4" (shape input) (at 73.66 134.62 0) (fields_autoplaced)
+    (effects (font (size 1.27 1.27)) (justify left))
+    (property "Intersheetrefs" "${INTERSHEET_REFS}" (at 82.4924 134.62 0)
       (effects (font (size 1.27 1.27)) (justify left) hide)
     )
@@
     )
   )
-  (global_label "Left" (shape input) (at 73.66 142.24 0) (fields_autoplaced)
-    (effects (font (size 1.27 1.27)) (justify left))
-    (property "Intersheetrefs" "${INTERSHEET_REFS}" (at 80.1339 142.24 0)
+  (global_label "Left" (shape input) (at 73.66 132.08 0) (fields_autoplaced)
+    (effects (font (size 1.27 1.27)) (justify left))
+    (property "Intersheetrefs" "${INTERSHEET_REFS}" (at 80.1339 132.08 0)
       (effects (font (size 1.27 1.27)) (justify left) hide)
     )
@@
     )
   )
-  (global_label "Col 9" (shape input) (at 73.66 127 0) (fields_autoplaced)
-    (effects (font (size 1.27 1.27)) (justify left))
-    (property "Intersheetrefs" "${INTERSHEET_REFS}" (at 81.8271 127 0)
-      (effects (font (size 1.27 1.27)) (justify left) hide)
-    )
+  (global_label "Col 9" (shape input) (at 73.66 139.7 0) (fields_autoplaced)
+    (effects (font (size 1.27 1.27)) (justify left))
+    (property "Intersheetrefs" "${INTERSHEET_REFS}" (at 81.8271 139.7 0)
+      (effects (font (size 1.27 1.27)) (justify left) hide)
+    )

Commit message: anya r2
Parts:
- removed D34, D35, D36: LED, LED_THT:LED_D3.0mm, symbol Device:LED
- removed R1, R3, R5: R, Resistor_SMD:R_0805_2012Metric_Pad1.20x1.40mm_HandSolder, symbol Device:R
- removed R2, R4, R6: R, Resistor_THT:R_Axial_DIN0207_L6.3mm_D2.5mm_P10.16mm_Horizontal, symbol Device:R
- added LED1, LED2, LED3: YS-SK6812MINI-E, Keyboard_JSA:YS-SK6812MINI-E, symbol kbd:YS-SK6812MINI-E
- D1, D10, D11, D12, D13, D14, D15, D16, D17, D18, D19, D2, D20, D21, D22, D23, D24, D25, D26, D27, D28, D29, D3, D30, D31, D32, D33, D4, D5, D6, D7, D8, D9: footprint Diode_SMD:D_SOD-123 -> Keyboard_JSA:D3_SMD_v2
Connections:
- net GND: now also LED1.3 (VSS), LED2.3 (VSS), LED3.3 (VSS)
- net VCC: now also LED1.1 (VDD), LED2.1 (VDD), LED3.1 (VDD)
- net Left: no longer names the net of U1.17 (A0/PF7)
- net Left: now also LED1.4 (DIN)
- net Middle: no longer names the net of U1.18 (A1/PF6)
- net Right: no longer names the net of U1.19 (A2/PF5)
- new net: LED1.2 (DOUT), LED2.4 (DIN)
- new net: LED2.2 (DOUT), LED3.4 (DIN)
- no-connect marks 2 -> 6
