File: Pragmatic56/Input.kicad_pcb (KiCad board)
At the start: 2 copper layers, 126.7 x 100.2 mm, 118 parts, among them J1 Conn_02x04_Odd_Even, SW1 SW_Push_45deg, SW10 SW_Push_45deg, SW11 SW_Push_45deg, SW12 SW_Push_45deg, SW13 SW_Push_45deg, SW14 SW_Push_45deg, SW15 SW_Push_45deg, SW16 SW_Push_45deg, SW17 SW_Push_45deg, SW18 SW_Push_45deg, SW19 SW_Push_45deg, SW2 SW_Push_45deg, SW20 SW_Push_45deg, SW21 SW_Push_45deg, SW22 SW_Push_45deg, SW23 SW_Push_45deg, SW24 SW_Push_45deg, SW25 SW_Push_45deg, SW26 SW_Push_45deg, SW27 SW_Push_45deg, SW28 SW_Push_45deg, SW29 SW_Push_45deg, SW3 SW_Push_45deg, SW30 SW_Push_45deg, SW31 SW_Push_45deg, SW32 SW_Push_45deg, SW33 SW_Push_45deg, SW34 SW_Push_45deg, SW35 SW_Push_45deg, SW36 SW_Push_45deg, SW37 SW_Push_45deg, SW38 SW_Push_45deg, SW39 SW_Push_45deg, SW4 SW_Push_45deg, SW40 SW_Push_45deg, SW41 SW_Push_45deg, SW42 SW_Push_45deg, SW43 SW_Push_45deg, SW44 SW_Push_45deg, SW45 SW_Push_45deg, SW46 SW_Push_45deg, SW47 SW_Push_45deg, SW48 SW_Push_45deg, SW5 SW_Push_45deg, SW51 SW_Push_45deg, SW52 SW_Push_45deg, SW53 SW_Push_45deg, SW54 SW_Push_45deg, SW55 SW_Push_45deg, SW56 SW_Push_45deg, SW57 SW_Push_45deg, SW58 SW_Push_45deg, SW6 SW_Push_45deg, SW7 SW_Push_45deg, SW8 SW_Push_45deg, SW9 SW_Push_45deg

Commit message: fix all Kicad 7 DRC
Parts:
- turned D21 to 180 degrees
- turned D9 to 180 degrees
Routing:
- net Row 2: track 144.8 -> 148.0 mm, vias 6 -> 7
- net Net-(D9-Pad2): track 9.95 -> 13.1 mm
- net C56: track 306.8 -> 303.7 mm
- net Net-(D21-Pad2): track 9.95 -> 13.0 mm
- net Row 1: track 120.3 -> 121.6 mm
Other:
- board text added: "Pragmatic 56 Duplex Matrix R1 2023-03"
- board text removed: "Pragmatic 56 Duplex Matrix R1 2023-02"

Commit message: validated
Parts:
- moved H4 1.12 mm to (120.5, 95.0)
- moved D54 0.57 mm to (116.8, 135.3)
- moved D55 0.55 mm to (116.8, 135.3)
Routing:
- net Row 1: track 121.6 -> 120.5 mm
- net Net-(D21-Pad2): track 13.0 -> 12.0 mm
- net Net-(D9-Pad2): track 13.1 -> 12.3 mm
- net Net-(D55-Pad2): track 13.0 -> 13.7 mm
Other:
- board size 126.7 x 100.2 mm -> 127.4 x 100.1 mm
- board text added: "Pragmatic 56 Duplex Matrix R2 2023-04"
- board text removed: "Pragmatic 56 Duplex Matrix R1 2023-03"

Commit message: tidy up
Parts:
- moved H2 42.0 mm to (234.5, 103.5)
- moved H3 34.2 mm to (168.0, 51.0)
- moved H1 20.0 mm to (168.0, 146.0)
- moved D54 14.8 mm to (131.5, 137.1), turned to 90 degrees
- moved D55 14.8 mm to (131.5, 137.1), turned to -90 degrees
- moved D51 7.74 mm to (171.0, 136.7), turned to -90 degrees
- moved D58 7.74 mm to (171.0, 136.7), turned to 90 degrees
- moved D53 7.11 mm to (134.0, 137.0), turned to -90 degrees
- moved D56 7.11 mm to (134.0, 137.0), turned to 90 degrees
- moved D52 7.11 mm to (153.0, 137.0), turned to 90 degrees
- moved D57 7.11 mm to (153.0, 137.0), turned to -90 degrees
- moved D1 2.50 mm to (225.0, 69.5)
- moved D12 2.50 mm to (225.0, 69.5)
- moved D13 2.50 mm to (225.0, 87.5)
- moved D24 2.50 mm to (225.0, 87.5)
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Routing:
- net Row 5: track 147.6 -> 137.7 mm
- net Net-(D54-Pad1): track 11.5 -> 6.97 mm
- net Net-(D55-Pad2): track 13.7 -> 9.46 mm
- net C12: track 298.7 -> 302.4 mm, vias 15 -> 14
- net Row 3: track 162.8 -> 160.1 mm
- net Row 1: track 120.5 -> 118.2 mm, vias 8 -> 7
- net Net-(D58-Pad1): track 9.95 -> 12.1 mm
- net C34: track 326.6 -> 328.7 mm, vias 17 -> 16
- net Net-(D56-Pad1): track 10.7 -> 12.3 mm
- net Net-(D51-Pad2): track 12.4 -> 10.9 mm
- net C56: track 303.7 -> 305.1 mm
- net Row 2: track 147.6 -> 146.2 mm
- net Row 4: track 178.9 -> 177.7 mm
Other:
- board size 127.4 x 100.1 mm -> 126.4 x 100.6 mm
- board text added: "Pragmatic 56 R3 2023-07"
- board text removed: "Pragmatic 56 Duplex Matrix R2 2023-04"
