File: Pragmatic60/Input.kicad_pcb (KiCad board)
At the start: 2 copper layers, 114 x 97 mm, 121 parts, among them J1 Conn_02x04_Odd_Even, SW1 SW_Push_45deg, SW10 SW_Push_45deg, SW11 SW_Push_45deg, SW12 SW_Push_45deg, SW13 SW_Push_45deg, SW14 SW_Push_45deg, SW15 SW_Push_45deg, SW16 SW_Push_45deg, SW17 SW_Push_45deg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

Commit message: 60A ready
Parts:
- moved J1 0.50 mm to (95.0, 36.5)
Routing:
- net Row 4: track 206.0 -> 206.8 mm
Other:
- board size 114 x 97 mm -> 114 x 96.5 mm
