File: Pragmatic36/MX/Input.kicad_pcb (KiCad board)
At the start: 2 copper layers, 108.2 x 85.4 mm, 78 parts, among them J1 Conn_02x04_Odd_Even, SW14 SW_Push_45deg, SW15 SW_Push_45deg, SW16 SW_Push_45deg, SW17 SW_Push_45deg, SW18 SW_Push_45deg, SW19 SW_Push_45deg, SW20 SW_Push_45deg, SW21 SW_Push_45deg, SW22 SW_Push_45deg, SW23 SW_Push_45deg, SW26 SW_Push_45deg, SW27 SW_Push_45deg, SW28 SW_Push_45deg, SW29 SW_Push_45deg, SW30 SW_Push_45deg, SW31 SW_Push_45deg, SW32 SW_Push_45deg, SW33 SW_Push_45deg, SW34 SW_Push_45deg, SW35 SW_Push_45deg, SW38 SW_Push_45deg, SW39 SW_Push_45deg, SW40 SW_Push_45deg, SW41 SW_Push_45deg, SW42 SW_Push_45deg, SW43 SW_Push_45deg, SW44 SW_Push_45deg, SW45 SW_Push_45deg, SW46 SW_Push_45deg, SW47 SW_Push_45deg, SW52 SW_Push_45deg, SW53 SW_Push_45deg, SW54 SW_Push_45deg, SW55 SW_Push_45deg, SW56 SW_Push_45deg, SW57 SW_Push_45deg

Commit message: MX 36 wrap up
Parts:
- moved REF** 5.50 mm to (170.5, 129.0)
Other:
- board text added: "Pragmatic 36A R1 2023-05"
- board text removed: "Pragmatic 42A R2 2023-05"
Changed lines of the file:
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@@
   )
   (footprint "Keyboard_JSA:OSHW-Logo2_7.3x6mm_Copper" (layer "B.Cu")
-    (at 176 129 180)
+    (at 170.5 129 180)
     (descr "Open Source Hardware Symbol")
     (tags "Logo Symbol OSHW")
@@
     (effects (font (size 1 1) (thickness 0.15)))
   )
-  (gr_text "Pragmatic 42A\nR2 2023-05" (at 176 129) (layer "F.SilkS")
+  (gr_text "Pragmatic 36A\nR1 2023-05" (at 171.5 129) (layer "F.SilkS")
     (effects (font (size 1.5 1.5) (thickness 0.2)))
   )
@@
     (effects (font (size 1.5 1.5) (thickness 0.2)))
   )
+  (dimension (type aligned) (layer "B.Cu")
+    (pts (xy 119 62.5) (xy 119 74))
+    (height 18)
+    (gr_text "11.5000 mm" (at 99.2 68.25 90) (layer "B.Cu")
+      (effects (font (size 1.5 1.5) (thickness 0.3)))
+    )
+    (format (prefix "") (suffix "") (units 3) (units_format 1) (precision 4))
+    (style (thickness 0.2) (arrow_length 1.27) (text_position_mode 0) (extension_height 0.58642) (extension_offset 0.5) keep_text_aligned)
+  )
+  (dimension (type aligned) (layer "Cmts.User")
+    (pts (xy 119 74) (xy 119 93))
+    (height 18)
+    (gr_text "19.0000 mm" (at 99.2 83.5 90) (layer "Cmts.User")
+      (effects (font (size 1.5 1.5) (thickness 0.3)))
+    )
+    (format (prefix "") (suffix "") (units 3) (units_format 1) (precision 4))
+    (style (thickness 0.2) (arrow_length 1.27) (text_position_mode 0) (extension_height 0.58642) (extension_offset 0.5) keep_text_aligned)
+  )
   (dimension (type aligned) (layer "Cmts.User")
