File: Pragmatic54/MX/Input.kicad_sch (KiCad schematic)
At the start: 109 parts, among them J1 Conn_02x04_Odd_Even, SW1 SW_Push_45deg, SW10 SW_Push_45deg, SW11 SW_Push_45deg, SW12 SW_Push_45deg, SW13 SW_Push_45deg, SW14 SW_Push_45deg, SW15 SW_Push_45deg, SW16 SW_Push_45deg, SW17 SW_Push_45deg, SW18 SW_Push_45deg, SW19 SW_Push_45deg, SW2 SW_Push_45deg, SW20 SW_Push_45deg, SW21 SW_Push_45deg, SW22 SW_Push_45deg, SW23 SW_Push_45deg, SW24 SW_Push_45deg, SW25 SW_Push_45deg, SW26 SW_Push_45deg, SW27 SW_Push_45deg, SW28 SW_Push_45deg, SW29 SW_Push_45deg, SW3 SW_Push_45deg, SW30 SW_Push_45deg, SW31 SW_Push_45deg, SW32 SW_Push_45deg, SW33 SW_Push_45deg, SW34 SW_Push_45deg, SW35 SW_Push_45deg, SW36 SW_Push_45deg, SW37 SW_Push_45deg, SW38 SW_Push_45deg, SW39 SW_Push_45deg, SW4 SW_Push_45deg, SW40 SW_Push_45deg, SW41 SW_Push_45deg, SW42 SW_Push_45deg, SW43 SW_Push_45deg, SW44 SW_Push_45deg, SW45 SW_Push_45deg, SW46 SW_Push_45deg, SW47 SW_Push_45deg, SW48 SW_Push_45deg, SW5 SW_Push_45deg, SW52 SW_Push_45deg, SW53 SW_Push_45deg, SW54 SW_Push_45deg, SW55 SW_Push_45deg, SW56 SW_Push_45deg, SW57 SW_Push_45deg, SW6 SW_Push_45deg, SW7 SW_Push_45deg, SW8 SW_Push_45deg, SW9 SW_Push_45deg

Commit message: MX54 R2.2 key switch on south
Connections:
- net C12: now also SW17.2, SW18.1, SW19.1, SW20.2, SW29.2, SW30.1, SW31.1, SW32.2, SW41.2, SW42.1, SW43.1, SW44.2, SW53.2, SW54.1, SW55.1, SW56.2; no longer SW17.1, SW18.2, SW19.2, SW20.1, SW29.1, SW30.2, SW31.2, SW32.1, SW41.1, SW42.2, SW43.2, SW44.1, SW53.1, SW54.2, SW55.2, SW56.1
- net C34: now also SW15.2, SW16.1, SW21.1, SW22.2, SW27.2, SW28.1, SW33.1, SW34.2, SW39.2, SW40.1, SW45.1, SW46.2, SW52.1, SW57.1; no longer SW15.1, SW16.2, SW21.2, SW22.1, SW27.1, SW28.2, SW33.2, SW34.1, SW39.1, SW40.2, SW45.2, SW46.1, SW52.2, SW57.2
- net C56: now also SW1.2, SW12.2, SW13.2, SW14.1, SW23.1, SW24.2, SW25.2, SW26.1, SW35.1, SW36.2, SW37.2, SW38.1, SW47.1, SW48.2; no longer SW1.1, SW12.1, SW13.1, SW14.2, SW23.2, SW24.1, SW25.1, SW26.2, SW35.2, SW36.1, SW37.1, SW38.2, SW47.2, SW48.1
- net at D21.2 (A): now also SW21.2; no longer SW21.1
- net at D25.2 (A): now also SW25.1; no longer SW25.2
- net at D37.2 (A): now also SW37.1; no longer SW37.2
- net at D14.1 (K): now also SW14.2; no longer SW14.1
- net at D33.2 (A): now also SW33.2; no longer SW33.1
- net at D19.2 (A): now also SW19.2; no longer SW19.1
- net at D54.1 (K): now also SW54.2; no longer SW54.1
- net at D43.2 (A): now also SW43.2; no longer SW43.1
- net at D45.2 (A): now also SW45.2; no longer SW45.1
- net at D28.1 (K): now also SW28.2; no longer SW28.1
- net at D17.2 (A): now also SW17.1; no longer SW17.2
- net at D15.2 (A): now also SW15.1; no longer SW15.2
- net at D20.1 (K): now also SW20.1; no longer SW20.2
- net at D41.2 (A): now also SW41.1; no longer SW41.2
- net at D13.2 (A): now also SW13.1; no longer SW13.2
- net at D27.2 (A): now also SW27.1; no longer SW27.2
- net at D36.1 (K): now also SW36.1; no longer SW36.2
- net at D35.2 (A): now also SW35.2; no longer SW35.1
- net at D32.1 (K): now also SW32.1; no longer SW32.2
- net at D38.1 (K): now also SW38.2; no longer SW38.1
- net at D31.2 (A): now also SW31.2; no longer SW31.1
- net at D40.1 (K): now also SW40.2; no longer SW40.1
- net at D24.1 (K): now also SW24.1; no longer SW24.2
- net at D55.2 (A): now also SW55.2; no longer SW55.1
- net at D52.1 (K): now also SW52.2; no longer SW52.1
- net at D48.1 (K): now also SW48.1; no longer SW48.2
- net at D22.1 (K): now also SW22.1; no longer SW22.2
- net at D12.1 (K): now also SW12.1; no longer SW12.2
- net at D56.1 (K): now also SW56.1; no longer SW56.2
- net at D30.1 (K): now also SW30.2; no longer SW30.1
- net at D42.1 (K): now also SW42.2; no longer SW42.1
- net at D46.1 (K): now also SW46.1; no longer SW46.2
- net at D18.1 (K): now also SW18.2; no longer SW18.1
- net at D39.2 (A): now also SW39.1; no longer SW39.2
- net at D57.2 (A): now also SW57.2; no longer SW57.1
- net at D26.1 (K): now also SW26.2; no longer SW26.1
- net at D47.2 (A): now also SW47.2; no longer SW47.1
- net at D29.2 (A): now also SW29.1; no longer SW29.2
- net at D34.1 (K): now also SW34.1; no longer SW34.2
- net at D1.2 (A): now also SW1.1; no longer SW1.2
- net at D44.1 (K): now also SW44.1; no longer SW44.2
- net at D53.2 (A): now also SW53.1; no longer SW53.2
- net at D16.1 (K): now also SW16.2; no longer SW16.1
- net at D23.2 (A): now also SW23.2; no longer SW23.1
Other:
- moved on the sheet: SW1, SW12, SW13, SW14, SW15, SW16, SW17, SW18, SW19, SW20, SW21, SW22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
