File: mx66/pcb/6666.kicad_pcb (KiCad board)
At the start: 2 copper layers, 371.7 x 95.2 mm, 145 parts, among them K1 100, K10 125, K11 100, K12 100, K13 100, K14 100, K15 125, K16 100, K17 100, K18 100, K19 100, K2 150, K20 125, K21 100, K22 100, K23 100, K24 100, K25 225, K26 100, K27 100, K28 100, K29 100, K3 175, K30 100, K31 100, K32 100, K33 100, K34 100, K35 100, K36 100, K37 100, K38 100, K39 100, K4 225, K40 100, K41 100, K42 100, K43 275, K44 100, K45 100, K46 100, K47 100, K48 125, K49 100, K5 125, K50 100, K51 100, K52 100, K53 125, K54 100, K55 100, K56 100, K57 100, K58 100, K59 100, K6 100, K60 100, K61 100, K62 200, K63 150, K64 225, K65 100, K66 100, K7 100, K8 100, K9 100, T1 AudioJack4, T2 AudioJack4, U1 MCU_ProMicro_13p, U2 MCU_ProMicro_13p

Commit message: add matrix.track
Parts:
- D1, D10, D11, D12, D13, D14, D15, D16, D17, D18, D19, D2, D20, D21, D22, D23, D24, D25, D26, D27, D28, D29, D3, D30, D31, D32, D33, D34, D35, D36, D37, D38, D39, D4, D40, D41, D42, D43, D44, D45, D46, D47, D48, D49, D5, D50, D51, D52, D53, D54, D55, D56, D57, D58, D59, D6, D60, D61, D62, D63, D64, D65, D66, D67, D7, D8, D9: footprint DreaM117er-keebLibrary:D_SOD-123 -> DreaM117er-keebLibrary:D_DO-35_SOD27_P7.62mm_Horizontal; moved to B.Cu
- moved D25 165.9 mm to (148.8, 182.3), turned to 90 degrees
- moved D48 158.9 mm to (311.0, 182.3), turned to 90 degrees
- moved D58 155.1 mm to (356.2, 182.3), turned to 90 degrees
- moved D43 154.0 mm to (272.9, 182.3), turned to 90 degrees
- moved D24 148.9 mm to (141.7, 163.2), turned to 90 degrees
- moved D38 148.4 mm to (280.0, 163.2), turned to 90 degrees
- moved D29 148.1 mm to (160.7, 163.2), turned to 90 degrees
- moved D67 144.6 mm to (394.3, 182.3), turned to 90 degrees
- moved D62 141.8 mm to (375.3, 182.3), turned to 90 degrees
- moved D47 141.8 mm to (318.1, 163.2), turned to 90 degrees
- moved D15 140.8 mm to (91.7, 182.3), turned to 90 degrees
- moved D57 139.4 mm to (356.2, 163.2), turned to 90 degrees
- moved D53 136.9 mm to (334.8, 182.3), turned to 90 degrees
- moved D34 136.6 mm to (261.0, 163.2), turned to 90 degrees
- moved D20 134.4 mm to (115.5, 182.3), turned to 90 degrees
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Connections:
- D1 pad 1: unconnected-(D1-Pad1) -> row0
- D10 pad 1: unconnected-(D10-Pad1) -> row4
- D11 pad 1: unconnected-(D11-Pad1) -> row0
- D12 pad 1: unconnected-(D12-Pad1) -> row1
- D13 pad 1: unconnected-(D13-Pad1) -> row2
- D14 pad 1: unconnected-(D14-Pad1) -> row3
- D15 pad 1: unconnected-(D15-Pad1) -> row4
- D16 pad 1: unconnected-(D16-Pad1) -> row0
- D17 pad 1: unconnected-(D17-Pad1) -> row1
- D18 pad 1: unconnected-(D18-Pad1) -> row2
- D19 pad 1: unconnected-(D19-Pad1) -> row3
- D2 pad 1: unconnected-(D2-Pad1) -> row1
- D20 pad 1: unconnected-(D20-Pad1) -> row4
- D21 pad 1: unconnected-(D21-Pad1) -> row0
- D22 pad 1: unconnected-(D22-Pad1) -> row1
- D23 pad 1: unconnected-(D23-Pad1) -> row2
- D24 pad 1: unconnected-(D24-Pad1) -> row3
- D25 pad 1: unconnected-(D25-Pad1) -> row4
- D26 pad 1: unconnected-(D26-Pad1) -> row0
- D27 pad 1: unconnected-(D27-Pad1) -> row1
- D28 pad 1: unconnected-(D28-Pad1) -> row2
- D29 pad 1: unconnected-(D29-Pad1) -> row3
- D3 pad 1: unconnected-(D3-Pad1) -> row2
- D30 pad 1: unconnected-(D30-Pad1) -> row0
- D31 pad 1: unconnected-(D31-Pad1) -> row5
- D32 pad 1: unconnected-(D32-Pad1) -> row6
- D33 pad 1: unconnected-(D33-Pad1) -> row7
- D34 pad 1: unconnected-(D34-Pad1) -> row8
- D35 pad 1: unconnected-(D35-Pad1) -> row5
- D36 pad 1: unconnected-(D36-Pad1) -> row6
- D37 pad 1: unconnected-(D37-Pad1) -> row7
- D38 pad 1: unconnected-(D38-Pad1) -> row8
- D39 pad 1: unconnected-(D39-Pad1) -> row5
- D4 pad 1: unconnected-(D4-Pad1) -> row3
- D40 pad 1: unconnected-(D40-Pad1) -> row6
- D41 pad 1: unconnected-(D41-Pad1) -> row7
- D42 pad 1: unconnected-(D42-Pad1) -> row8
- D43 pad 1: unconnected-(D43-Pad1) -> row9
- D44 pad 1: unconnected-(D44-Pad1) -> row5
- D45 pad 1: unconnected-(D45-Pad1) -> row6
- D46 pad 1: unconnected-(D46-Pad1) -> row7
- D47 pad 1: unconnected-(D47-Pad1) -> row8
- D48 pad 1: unconnected-(D48-Pad1) -> row9
- D49 pad 1: unconnected-(D49-Pad1) -> row5
- D5 pad 1: unconnected-(D5-Pad1) -> row4
- D50 pad 1: unconnected-(D50-Pad1) -> row6
- D51 pad 1: unconnected-(D51-Pad1) -> row7
- D52 pad 1: unconnected-(D52-Pad1) -> row8
- D53 pad 1: unconnected-(D53-Pad1) -> row9
- D54 pad 1: unconnected-(D54-Pad1) -> row5
- D55 pad 1: unconnected-(D55-Pad1) -> row6
- D56 pad 1: unconnected-(D56-Pad1) -> row7
- D57 pad 1: unconnected-(D57-Pad1) -> row8
- D58 pad 1: unconnected-(D58-Pad1) -> row9
- D59 pad 1: unconnected-(D59-Pad1) -> row5
- D6 pad 1: unconnected-(D6-Pad1) -> row0
- D60 pad 1: unconnected-(D60-Pad1) -> row6
- D61 pad 1: unconnected-(D61-Pad1) -> row8
- D62 pad 1: unconnected-(D62-Pad1) -> row9
- D63 pad 1: unconnected-(D63-Pad1) -> row5
- D64 pad 1: unconnected-(D64-Pad1) -> row6
- D65 pad 1: unconnected-(D65-Pad1) -> row7
- D66 pad 1: unconnected-(D66-Pad1) -> row8
- D67 pad 1: unconnected-(D67-Pad1) -> row9
- D7 pad 1: unconnected-(D7-Pad1) -> row1
- D8 pad 1: unconnected-(D8-Pad1) -> row2
- D9 pad 1: unconnected-(D9-Pad1) -> row3
- K1 pad 1: unconnected-(K1-Pad1) -> col0.L
- K10 pad 1: unconnected-(K10-Pad1) -> col1.L
- K11 pad 1: unconnected-(K11-Pad1) -> col2.L
- K12 pad 1: unconnected-(K12-Pad1) -> col2.L
- K13 pad 1: unconnected-(K13-Pad1) -> col2.L
- K14 pad 1: unconnected-(K14-Pad1) -> col2.L
- K15 pad 1: unconnected-(K15-Pad1) -> col2.L
- K16 pad 1: unconnected-(K16-Pad1) -> col3.L
- K17 pad 1: unconnected-(K17-Pad1) -> col3.L
- K18 pad 1: unconnected-(K18-Pad1) -> col3.L
- K19 pad 1: unconnected-(K19-Pad1) -> col3.L
- K2 pad 1: unconnected-(K2-Pad1) -> col0.L
- K20 pad 1: unconnected-(K20-Pad1) -> col3.L
- K21 pad 1: unconnected-(K21-Pad1) -> col4.L
- K22 pad 1: unconnected-(K22-Pad1) -> col4.L
- K23 pad 1: unconnected-(K23-Pad1) -> col4.L
- K24 pad 1: unconnected-(K24-Pad1) -> col4.L
- K25 pad 1: unconnected-(K25-Pad1) -> col4.L
- K26 pad 1: unconnected-(K26-Pad1) -> col5.L
- K27 pad 1: unconnected-(K27-Pad1) -> col5.L
- K28 pad 1: unconnected-(K28-Pad1) -> col5.L
- K29 pad 1: unconnected-(K29-Pad1) -> col5.L
- K3 pad 1: unconnected-(K3-Pad1) -> Net-(D3-Pad2)
- K3 pad 2: Net-(D3-Pad2) -> col0.L
- K30 pad 1: unconnected-(K30-Pad1) -> col6.L
- K31 pad 1: unconnected-(K31-Pad1) -> col7.R
- K32 pad 1: unconnected-(K32-Pad1) -> col7.R
- K33 pad 1: unconnected-(K33-Pad1) -> col7.R
- K34 pad 1: unconnected-(K34-Pad1) -> col7.R
- K35 pad 1: unconnected-(K35-Pad1) -> col6.R
- K36 pad 1: unconnected-(K36-Pad1) -> col6.R
- K37 pad 1: unconnected-(K37-Pad1) -> col6.R
- K38 pad 1: unconnected-(K38-Pad1) -> col6.R
- K39 pad 1: unconnected-(K39-Pad1) -> col5.R
- K4 pad 1: unconnected-(K4-Pad1) -> col0.L
- K40 pad 1: unconnected-(K40-Pad1) -> col5.R
- K41 pad 1: unconnected-(K41-Pad1) -> col5.R
- K42 pad 1: unconnected-(K42-Pad1) -> col5.R
- K43 pad 1: unconnected-(K43-Pad1) -> col6.R
- K44 pad 1: unconnected-(K44-Pad1) -> col4.R
- K45 pad 1: unconnected-(K45-Pad1) -> col4.R
- K46 pad 1: unconnected-(K46-Pad1) -> col4.R
- K47 pad 1: unconnected-(K47-Pad1) -> col4.R
- K48 pad 1: unconnected-(K48-Pad1) -> col4.R
- K49 pad 1: unconnected-(K49-Pad1) -> col3.R
- K5 pad 1: unconnected-(K5-Pad1) -> col0.L
- K50 pad 1: unconnected-(K50-Pad1) -> col3.R
- K51 pad 1: unconnected-(K51-Pad1) -> col3.R
- K52 pad 1: unconnected-(K52-Pad1) -> col3.R
- K53 pad 1: unconnected-(K53-Pad1) -> col3.R
- K54 pad 1: unconnected-(K54-Pad1) -> col2.R
- K55 pad 1: unconnected-(K55-Pad1) -> col2.R
- K56 pad 1: unconnected-(K56-Pad1) -> col2.R
- K57 pad 1: unconnected-(K57-Pad1) -> col2.R
- K58 pad 1: unconnected-(K58-Pad1) -> col2.R
- K59 pad 1: unconnected-(K59-Pad1) -> col1.R
- K6 pad 1: unconnected-(K6-Pad1) -> col1.L
- K60 pad 1: unconnected-(K60-Pad1) -> col1.R
- K61 pad 1: unconnected-(K61-Pad1) -> col1.R
- K62 pad 1: unconnected-(K62-Pad1) -> Net-(D59-Pad2)
- K62 pad 2: Net-(D63-Pad2) -> col1.R
- K63 pad 1: unconnected-(K63-Pad1) -> col0.R
- K64 pad 1: unconnected-(K64-Pad1) -> col0.R
- K65 pad 1: unconnected-(K65-Pad1) -> col0.R
- K66 pad 1: unconnected-(K66-Pad1) -> col0.R
- K7 pad 1: unconnected-(K7-Pad1) -> col1.L
- K8 pad 1: unconnected-(K8-Pad1) -> col1.L
- K9 pad 1: unconnected-(K9-Pad1) -> col1.L
- O1 pad 1: unconnected-(O1-Pad1) -> col0.L
- O2 pad 1: unconnected-(O2-Pad1) -> Net-(D59-Pad2)
- O2 pad 2: Net-(D59-Pad2) -> col1.R
- O3 pad 1: unconnected-(O3-Pad1) -> Net-(D63-Pad2)
- O3 pad 2: Net-(D63-Pad2) -> col0.R
Routing:
- net row6: track 0.00 -> 155.3 mm
- net row8: track 0.00 -> 150.6 mm
- net row7: track 0.00 -> 142.8 mm
- net row5: track 0.00 -> 137.5 mm
- net row9: track 0.00 -> 136.0 mm
- net row0: track 0.00 -> 129.4 mm
- net row3: track 0.00 -> 121.0 mm
- net row4: track 0.00 -> 117.2 mm
- net row2: track 0.00 -> 113.3 mm
- net row1: track 0.00 -> 110.8 mm
- net col1.R: track 0.00 -> 102.0 mm
- net col1.L: track 0.00 -> 93.9 mm
- net col2.L: track 0.00 -> 91.9 mm
- net col4.L: track 0.00 -> 87.2 mm
- net col3.L: track 0.00 -> 87.2 mm
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
Commit message: re-put footprint and newtrack
Parts:
- removed T1, T2: AudioJack4, DreaM117er-keebLibrary:TRRS-PJ-320A
- added J1: Left side, DreaM117er-keebLibrary:TRRS-PJ-320A, F.Cu at (181.5, 183.3)
- added J2: Right side, DreaM117er-keebLibrary:TRRS-PJ-320A, F.Cu at (215.0, 183.3)
- K1, K11, K12, K13, K14, K16, K17, K18, K19, K21, K22, K23, K24, K26, K27, K28, K29, K30, K31, K32, K33, K34, K35, K36, K37, K38, K39, K40, K41, K42, K44, K45, K46, K47, K49, K50, K51, K52, K54, K55, K56, K57, K58, K59, K6, K60, K61, K65, K66, K7, K8, K9, O2, O3: footprint DreaM117er-keebLibrary:SW_Hotswap_Kailh_MX_Plated_1.00u -> PCM_Switch_Keyboard_Hotswap_Kailh:SW_Hotswap_Kailh_MX_1.00u
- K10, K15, K20, K48, K5, K53, O1: footprint DreaM117er-keebLibrary:SW_Hotswap_Kailh_MX_Plated_1.25u -> PCM_Switch_Keyboard_Hotswap_Kailh:SW_Hotswap_Kailh_MX_1.25u
- K2, K63: footprint DreaM117er-keebLibrary:SW_Hotswap_Kailh_MX_Plated_1.50u -> PCM_Switch_Keyboard_Hotswap_Kailh:SW_Hotswap_Kailh_MX_1.50u
- K25, K4, K64: footprint DreaM117er-keebLibrary:SW_Hotswap_Kailh_MX_Plated_2.25u -> PCM_Switch_Keyboard_Hotswap_Kailh:SW_Hotswap_Kailh_MX_2.25u
- K3: footprint DreaM117er-keebLibrary:SW_Hotswap_Kailh_MX_Plated_1.75u -> PCM_Switch_Keyboard_Hotswap_Kailh:SW_Hotswap_Kailh_MX_1.75u
- K43: footprint DreaM117er-keebLibrary:SW_Hotswap_Kailh_MX_Plated_2.75u -> PCM_Switch_Keyboard_Hotswap_Kailh:SW_Hotswap_Kailh_MX_2.75u
- K62: footprint DreaM117er-keebLibrary:SW_Hotswap_Kailh_MX_Plated_2.00u -> PCM_Switch_Keyboard_Hotswap_Kailh:SW_Hotswap_Kailh_MX_2.00u
- turned stab4 to 0 degrees
Connections:
- K25 pad 1: col4.L -> col5.L
- O2 pad 1: Net-(D59-Pad2) -> col1.R
- O2 pad 2: col1.R -> Net-(D59-Pad2)
- U1 pad 2: unconnected-(U1-0/PD3-Pad2) -> TX-L
- U1 pad 22: unconnected-(U1-VCC-Pad22) -> VCC-L
- U1 pad 24: unconnected-(U1-GND-Pad24) -> GND-L
- U1 pad 3: unconnected-(U1-1/PD2-Pad3) -> RX-L
- U1 pad 4: unconnected-(U1-GND-Pad4) -> GND-L
- U1 pad 5: unconnected-(U1-GND-Pad5) -> GND-L
- U2 pad 2: unconnected-(U2-0/PD3-Pad2) -> TX-R
- U2 pad 22: unconnected-(U2-VCC-Pad22) -> VCC-R
- U2 pad 24: unconnected-(U2-GND-Pad24) -> GND-R
- U2 pad 3: unconnected-(U2-1/PD2-Pad3) -> RX-R
- U2 pad 4: unconnected-(U2-GND-Pad4) -> GND-R
- U2 pad 5: unconnected-(U2-GND-Pad5) -> GND-R
Routing:
- net col5.L: track 66.3 -> 109.8 mm
- net col1.L: track 93.9 -> 114.6 mm
- net col2.L: track 91.9 -> 109.8 mm
- net col3.L: track 87.2 -> 105.0 mm
- net row8: track 150.6 -> 133.4 mm
- net row6: track 155.3 -> 138.1 mm
- net col4.R: track 83.8 -> 100.3 mm
- net col6.R: track 83.8 -> 100.3 mm
- net col0.L: track 83.6 -> 99.9 mm
- net row5: track 137.5 -> 122.0 mm
- net col1.R: track 102.0 -> 117.3 mm
- net row0: track 129.4 -> 114.3 mm
- net row7: track 142.8 -> 127.9 mm
- net row2: track 113.3 -> 100.4 mm
- net row9: track 136.0 -> 123.1 mm
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
Commit message: re-put footprint and newtrack
Routing:
- net Net-(D3-Pad2): track 16.4 -> 18.6 mm
- net Net-(D59-Pad2): track 21.8 -> 22.4 mm
Changed lines of the file:
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@@
 			(net 67 "unconnected-(U1-?-Pad1)")
 			(pinfunction "?")
-			(pintype "passive")
+			(pintype "passive+no_connect")
 		)
 		(pad "2" thru_hole circle
@@
 			(net 71 "unconnected-(U1-?-Pad26)")
 			(pinfunction "?")
-			(pintype "passive")
+			(pintype "passive+no_connect")
 		)
 		(embedded_fonts no)
@@
 			(net 87 "unconnected-(U2-?-Pad1)")
 			(pinfunction "?")
-			(pintype "passive")
+			(pintype "passive+no_connect")
 		)
 		(pad "2" thru_hole circle
@@
 			(net 93 "unconnected-(U2-?-Pad26)")
 			(pinfunction "?")
-			(pintype "passive")
+			(pintype "passive+no_connect")
 		)
 		(embedded_fonts no)
@@
 	)
 	(segment
-		(start 50.80375 143.36625)
-		(end 50.34 143.83)
+		(start 42.097 136.165)
+		(end 50.345 136.165)
 		(width 0.5)
 		(layer "B.Cu")
@@
 	)
 	(segment
-		(start 50.34 143.83)
-		(end 48.08875 143.83)
+		(start 48.08875 143.83)
+		(end 48.08875 140.84125)
 		(width 0.5)
 		(layer "B.Cu")
@@
 	)
 	(segment
-		(start 42.097 136.165)
-		(end 50.345 136.165)
+		(start 48.54 140.39)
+		(end 50.80375 140.39)
 		(width 0.5)
 		(layer "B.Cu")
@@
 	)
 	(segment
-		(start 50.80375 142.54)
-		(end 50.80375 143.36625)
+		(start 50.80375 136.62375)
+		(end 50.80375 140.39)
 		(width 0.5)
 		(layer "B.Cu")
@@
 	)
 	(segment
-		(start 50.80375 136.62375)
-		(end 50.80375 140.39)
+		(start 48.08875 140.84125)
+		(end 48.54 140.39)
 		(width 0.5)
 		(layer "B.Cu")
@@
 	)
 	(segment
-		(start 361.618 108.27)
-		(end 361.618 105.532)
+		(start 364.36 104.6)
+		(end 364.36 99.1)
 		(width 0.5)
 		(layer "B.Cu")
@@
 	)
 	(segment
-		(start 360.11 100.65)
-		(end 364.36 100.65)
+		(start 359.66 98.64)
+		(end 363.9 98.64)
 		(width 0.5)
 		(layer "B.Cu")
@@
 	)
 	(segment
-		(start 362.08 105.07)
-		(end 363.89 105.07)
+		(start 361.618 105.532)
+		(end 362.08 105.07)
 		(width 0.5)
 		(layer "B.Cu")
@@
 	)
 	(segment
-		(start 360.11 100.65)
-		(end 359.66 100.2)
+		(start 363.89 105.07)
+		(end 364.36 104.6)
 		(width 0.5)
 		(layer "B.Cu")
@@
 	)
 	(segment
-		(start 363.89 105.07)
-		(end 364.36 104.6)
+		(start 364.36 99.1)
+		(end 368.35 99.1)
 		(width 0.5)
 		(layer "B.Cu")
@@
 	)
 	(segment
-		(start 361.618 105.532)
-		(end 362.08 105.07)
+		(start 361.618 108.27)
+		(end 361.618 105.532)
 		(width 0.5)
 		(layer "B.Cu")
@@
 	)
 	(segment
-		(start 359.66 100.2)
-		(end 359.66 98.64)
+		(start 363.9 98.64)
+		(end 364.36 99.1)
 		(width 0.5)
 		(layer "B.Cu")
@@
 	)
 	(segment
-		(start 364.36 100.65)
+		(start 368.35 99.1)
 		(end 369.9 100.65)
 		(width 0.5)
@@
 	)
 	(segment
-		(start 364.36 104.6)
-		(end 364.36 100.65)
+		(start 362.08 105.07)
+		(end 363.89 105.07)
 		(width 0.5)
 		(layer "B.Cu")
@@
 		(start 350.85 119.7)
 		(end 350.85 131.31)
-		(width 0.2)
+		(width 0.5)
 		(layer "B.Cu")
 		(net 135)

Commit message: set pinout and layout
Parts:
- added J10: OLED, DreaM117er-keebLibrary:PinHeader_1x04_P2.54mm_Vertical, F.Cu at (220.9, 132.6)
- added J3: Left side, DreaM117er-keebLibrary:TRRS-PJ-320A, F.Cu at (185.2, 93.8)
- added J4: Left side, DreaM117er-keebLibrary:TRRS-PJ-320A, F.Cu at (189.6, 141.3)
- added J5: Right side, DreaM117er-keebLibrary:TRRS-PJ-320A, F.Cu at (211.3, 93.8)
- added J6: Right side, DreaM117er-keebLibrary:TRRS-PJ-320A, F.Cu at (207.0, 141.3)
- added J7: Battery PH2.0, Connector_JST:JST_PH_S2B-PH-K_1x02_P2.00mm_Horizontal, F.Cu at (171.2, 196.0)
- added J8: Battery PH2.0, Connector_JST:JST_PH_S2B-PH-K_1x02_P2.00mm_Horizontal, F.Cu at (220.0, 196.5)
- added J9: OLED, DreaM117er-keebLibrary:PinHeader_1x04_P2.54mm_Vertical, F.Cu at (168.1, 132.6)
- added SW1: RST-L, DreaM117er-keebLibrary:ResetSW_1side, F.Cu at (188.0, 132.6)
- added SW2: RST-R, DreaM117er-keebLibrary:ResetSW_1side, F.Cu at (208.6, 132.6)
- U1, U2: moved to B.Cu
- moved J1 8.03 mm to (189.6, 183.3)
- moved J2 8.02 mm to (207.0, 183.3)
- turned U1 to 180 degrees
- turned U2 to 180 degrees
Connections:
- J1 pad R1: RX-L -> Data-L
- J1 pad R2: TX-L -> GND-L
- J1 pad S: GND-L -> unconnected-(J1-PadS)
- J2 pad R1: RX-R -> Data-R
- J2 pad R2: TX-R -> GND-R
- J2 pad S: GND-R -> unconnected-(J2-PadS)
- U1 pad 1: unconnected-(U1-?-Pad1) -> GND-L
- U1 pad 10: unconnected-(U1-6/PD7-Pad10) -> row1
- U1 pad 11: unconnected-(U1-7/PE6-Pad11) -> row2
- U1 pad 12: unconnected-(U1-8/PB4-Pad12) -> row3
- U1 pad 13: unconnected-(U1-9/PB5-Pad13) -> row4
- U1 pad 15: unconnected-(U1-23/PB2-Pad15) -> col6.L
- U1 pad 16: unconnected-(U1-20/PB3-Pad16) -> col5.L
- U1 pad 17: unconnected-(U1-22/PB1-Pad17) -> col4.L
- U1 pad 18: unconnected-(U1-26/PF7-Pad18) -> col3.L
- U1 pad 19: unconnected-(U1-27/PF6-Pad19) -> col2.L
- U1 pad 2: TX-L -> Data-L
- U1 pad 20: unconnected-(U1-28/PF5-Pad20) -> col1.L
- U1 pad 21: unconnected-(U1-29/PF4-Pad21) -> col0.L
- U1 pad 23: unconnected-(U1-RST-Pad23) -> RST-L
- U1 pad 25: unconnected-(U1-B0-Pad25) -> BAT+L
- U1 pad 26: unconnected-(U1-?-Pad26) -> BAT+L
- U1 pad 3: RX-L -> unconnected-(U1-1/PD2-Pad3)
- U1 pad 6: unconnected-(U1-2/PD1-Pad6) -> SDA-L
- U1 pad 7: unconnected-(U1-3/PD0-Pad7) -> SCL-L
- U1 pad 9: unconnected-(U1-5/PC6-Pad9) -> row0
- U2 pad 1: unconnected-(U2-?-Pad1) -> GND-R
- U2 pad 10: unconnected-(U2-6/PD7-Pad10) -> row6
- U2 pad 11: unconnected-(U2-7/PE6-Pad11) -> row7
- U2 pad 12: unconnected-(U2-8/PB4-Pad12) -> row8
- U2 pad 13: unconnected-(U2-9/PB5-Pad13) -> row9
- U2 pad 14: unconnected-(U2-21/PB6-Pad14) -> col7.R
- U2 pad 15: unconnected-(U2-23/PB2-Pad15) -> col6.R
- U2 pad 16: unconnected-(U2-20/PB3-Pad16) -> col5.R
- U2 pad 17: unconnected-(U2-22/PB1-Pad17) -> col4.R
- U2 pad 18: unconnected-(U2-26/PF7-Pad18) -> col3.R
- U2 pad 19: unconnected-(U2-27/PF6-Pad19) -> col2.R
- U2 pad 2: TX-R -> Data-R
- U2 pad 20: unconnected-(U2-28/PF5-Pad20) -> col1.R
- U2 pad 21: unconnected-(U2-29/PF4-Pad21) -> col0.R
- U2 pad 23: unconnected-(U2-RST-Pad23) -> RST-R
- U2 pad 25: unconnected-(U2-B0-Pad25) -> BAT+R
- U2 pad 26: unconnected-(U2-?-Pad26) -> BAT+R
- U2 pad 3: RX-R -> unconnected-(U2-1/PD2-Pad3)
- U2 pad 6: unconnected-(U2-2/PD1-Pad6) -> SDA-R
- U2 pad 7: unconnected-(U2-3/PD0-Pad7) -> SCL-R
- U2 pad 9: unconnected-(U2-5/PC6-Pad9) -> row5
Other:
- outline, holes or cut-outs redrawn

Commit message: finish track and zone
Parts:
- added SW3: ON-OFF, Button_Switch_THT:SW_Slide_SPDT_Angled_CK_OS102011MA1Q, F.Cu at (187.3, 119.6)
- added SW4: ON-OFF, Button_Switch_THT:SW_Slide_SPDT_Angled_CK_OS102011MA1Q, F.Cu at (209.3, 115.6)
- moved J7 50.3 mm to (185.1, 147.6)
- moved J8 49.5 mm to (209.5, 148.1)
Connections:
- J7 pad 1: BAT+L -> Net-(J7-Pin_1)
- J8 pad 1: BAT+R -> Net-(J8-Pin_1)
Routing:
- net col0.R: track 91.8 -> 265.3 mm, vias 0 -> 1
- net col0.L: track 99.9 -> 268.2 mm, vias 0 -> 1
- net col1.R: track 117.3 -> 276.3 mm, vias 0 -> 1
- net col2.R: track 93.6 -> 231.6 mm, vias 0 -> 1
- net VCC-L: track 0.00 -> 136.1 mm, vias 0 -> 3
- net col1.L: track 114.6 -> 248.2 mm, vias 0 -> 1
- net col3.R: track 95.5 -> 212.2 mm, vias 0 -> 1
- net col2.L: track 109.8 -> 220.6 mm, vias 0 -> 1
- net row4: track 106.5 -> 212.5 mm, vias 0 -> 1
- net Data-R: track 0.00 -> 104.5 mm, vias 0 -> 1
- net Data-L: track 0.00 -> 103.9 mm
- net row9: track 123.1 -> 222.5 mm, vias 0 -> 1
- net VCC-R: track 0.00 -> 97.3 mm, vias 0 -> 1
- net col4.R: track 100.3 -> 195.8 mm, vias 0 -> 1
- net col3.L: track 105.0 -> 192.9 mm, vias 0 -> 1
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- added copper zone on B.Cu, net GND-L
- added copper zone on F.Cu, net GND-L
- added copper zone on B.Cu, net GND-R
- added copper zone on F.Cu, net GND-R

Commit message: fix TRRS and SlideSW
Parts:
- SW3, SW4: value ON-OFF -> OFF-ON
Connections:
- J1 pad R2: GND-L -> unconnected-(J1-PadR2)
- J1 pad S: unconnected-(J1-PadS) -> GND-L
- J2 pad R2: GND-R -> unconnected-(J2-PadR2)
- J2 pad S: unconnected-(J2-PadS) -> GND-R
- J3 pad R2: GND-L -> unconnected-(J3-PadR2)
- J3 pad S: unconnected-(J3-PadS) -> GND-L
- J4 pad R2: GND-L -> unconnected-(J4-PadR2)
- J4 pad S: unconnected-(J4-PadS) -> GND-L
- J5 pad R2: GND-R -> unconnected-(J5-PadR2)
- J5 pad S: unconnected-(J5-PadS) -> GND-R
- J6 pad R2: GND-R -> unconnected-(J6-PadR2)
- J6 pad S: unconnected-(J6-PadS) -> GND-R
- SW3 pad 1: Net-(J7-Pin_1) -> unconnected-(SW3-Pad1)
- SW3 pad 3: unconnected-(SW3-Pad3) -> Net-(J7-Pin_1)
- SW4 pad 1: unconnected-(SW4-Pad1) -> Net-(J8-Pin_1)
- SW4 pad 3: Net-(J8-Pin_1) -> unconnected-(SW4-Pad3)
Routing:
- net Net-(J7-Pin_1): track 30.9 -> 36.3 mm
- net Net-(J8-Pin_1): track 32.9 -> 36.7 mm
- net BAT+L: vias 1 -> 0
