File: mx66/pcb/6666.kicad_sch (KiCad schematic)
At the start: 145 parts, among them K1 100, K10 125, K11 100, K12 100, K13 100, K14 100, K15 125, K16 100, K17 100, K18 100, K19 100, K2 150, K20 125, K21 100, K22 100, K23 100, K24 100, K25 225, K26 100, K27 100, K28 100, K29 100, K3 175, K30 100, K31 100, K32 100, K33 100, K34 100, K35 100, K36 100, K37 100, K38 100, K39 100, K4 225, K40 100, K41 100, K42 100, K43 275, K44 100, K45 100, K46 100, K47 100, K48 125, K49 100, K5 125, K50 100, K51 100, K52 100, K53 125, K54 100, K55 100, K56 100, K57 100, K58 100, K59 100, K6 100, K60 100, K61 100, K62 200, K63 150, K64 225, K65 100, K66 100, K7 100, K8 100, K9 100, T1 AudioJack4, T2 AudioJack4, U1 MCU_ProMicro_13p, U2 MCU_ProMicro_13p

Commit message: add matrix.track
Parts:
- D1, D10, D11, D12, D13, D14, D15, D16, D17, D18, D19, D2, D20, D21, D22, D23, D24, D25, D26, D27, D28, D29, D3, D30, D31, D32, D33, D34, D35, D36, D37, D38, D39, D4, D40, D41, D42, D43, D44, D45, D46, D47, D48, D49, D5, D50, D51, D52, D53, D54, D55, D56, D57, D58, D59, D6, D60, D61, D62, D63, D64, D65, D66, D67, D7, D8, D9: footprint DreaM117er-keebLibrary:D_SOD-123 -> DreaM117er-keebLibrary:D_DO-35_SOD27_P7.62mm_Horizontal
Connections:
- net row5: now reaches D31.1
- net row5: now also D35.1, D39.1, D44.1, D49.1, D54.1, D59.1, D63.1
- net col0.R: now reaches K64.1
- net col0.R: now also K63.1, K65.1, K66.1, O3.2
- net col2.L: now reaches K12.1
- net col2.L: now also K11.1, K13.1, K14.1, K15.1
- net row3: now reaches D4.1
- net row3: now also D14.1, D19.1, D24.1, D29.1, D9.1
- net row6: now reaches D45.1
- net row6: now also D32.1, D36.1, D40.1, D50.1, D55.1, D60.1, D64.1
- net row4: now reaches D10.1
- net row4: now also D15.1, D20.1, D25.1, D5.1
- net col6.R: now reaches K35.1
- net col6.R: now also K36.1, K37.1, K38.1, K43.1
- net col5.L: now reaches K29.1
- net col5.L: now also K26.1, K27.1, K28.1
- net row9: now reaches D53.1
- net row9: now also D43.1, D48.1, D58.1, D62.1, D67.1
- net col3.L: now reaches K17.1
- net col3.L: now also K16.1, K18.1, K19.1, K20.1
- net col5.R: now reaches K42.1
- net col5.R: now also K39.1, K40.1, K41.1
- net at O2.1: now also D59.2, K62.1
- net col1.R: now reaches O2.2
- net col1.R: now also K59.1, K60.1, K61.1, K62.2; no longer D59.2
- net row7: now reaches D51.1
- net row7: now also D33.1, D37.1, D41.1, D46.1, D56.1, D65.1
- net col4.R: now reaches K45.1
- net col4.R: now also K44.1, K46.1, K47.1, K48.1
- net col0.L: now reaches K4.1
- net col0.L: now also K1.1, K2.1, K3.2, K5.1, O1.1
- net col4.L: now reaches K22.1
- net col4.L: now also K21.1, K23.1, K24.1, K25.1
- net row8: now reaches D61.1
- net row8: now also D34.1, D38.1, D42.1, D47.1, D52.1, D57.1, D66.1
- net row1: now reaches D27.1
- net row1: now also D12.1, D17.1, D2.1, D22.1, D7.1
- net row2: now reaches D28.1
- net row2: now also D13.1, D18.1, D23.1, D3.1, D8.1
- net col1.L: now reaches K9.1
- net col1.L: now also K10.1, K6.1, K7.1, K8.1
- net col3.R: now reaches K53.1
- net col3.R: now also K49.1, K50.1, K51.1, K52.1
- net row0: now reaches D11.1
- net row0: now also D1.1, D16.1, D21.1, D26.1, D30.1, D6.1
- net col2.R: now reaches K58.1
- net col2.R: now also K54.1, K55.1, K56.1, K57.1
- net col7.R: now reaches K32.1
- net col7.R: now also K31.1, K33.1, K34.1
- net at O3.1: now also D63.2
- net at D3.2, O1.2: now also K3.1; no longer K3.2
- net col6.L: now reaches K30.1
Other:
- moved on the sheet: D43, K3, K43, K62, O2, O3

Commit message: re-put footprint and newtrack
Parts:
- removed T1, T2: AudioJack4, DreaM117er-keebLibrary:TRRS-PJ-320A, symbol DreaM117er_Library:TRRS
- added J1: Left side, DreaM117er-keebLibrary:TRRS-PJ-320A, symbol Connector_Audio:AudioJack4
- added J2: Right side, DreaM117er-keebLibrary:TRRS-PJ-320A, symbol Connector_Audio:AudioJack4
- K1, K11, K12, K13, K14, K16, K17, K18, K19, K21, K22, K23, K24, K26, K27, K28, K29, K30, K31, K32, K33, K34, K35, K36, K37, K38, K39, K40, K41, K42, K44, K45, K46, K47, K49, K50, K51, K52, K54, K55, K56, K57, K58, K59, K6, K60, K61, K65, K66, K7, K8, K9, O2, O3: footprint DreaM117er-keebLibrary:SW_Hotswap_Kailh_MX_Plated_1.00u -> PCM_Switch_Keyboard_Hotswap_Kailh:SW_Hotswap_Kailh_MX_1.00u
- K10, K15, K20, K48, K5, K53, O1: footprint DreaM117er-keebLibrary:SW_Hotswap_Kailh_MX_Plated_1.25u -> PCM_Switch_Keyboard_Hotswap_Kailh:SW_Hotswap_Kailh_MX_1.25u
- K2, K63: footprint DreaM117er-keebLibrary:SW_Hotswap_Kailh_MX_Plated_1.50u -> PCM_Switch_Keyboard_Hotswap_Kailh:SW_Hotswap_Kailh_MX_1.50u
- K25, K4, K64: footprint DreaM117er-keebLibrary:SW_Hotswap_Kailh_MX_Plated_2.25u -> PCM_Switch_Keyboard_Hotswap_Kailh:SW_Hotswap_Kailh_MX_2.25u
- K3: footprint DreaM117er-keebLibrary:SW_Hotswap_Kailh_MX_Plated_1.75u -> PCM_Switch_Keyboard_Hotswap_Kailh:SW_Hotswap_Kailh_MX_1.75u
- K43: footprint DreaM117er-keebLibrary:SW_Hotswap_Kailh_MX_Plated_2.75u -> PCM_Switch_Keyboard_Hotswap_Kailh:SW_Hotswap_Kailh_MX_2.75u
- K62: footprint DreaM117er-keebLibrary:SW_Hotswap_Kailh_MX_Plated_2.00u -> PCM_Switch_Keyboard_Hotswap_Kailh:SW_Hotswap_Kailh_MX_2.00u
Connections:
- net col1.R: now also O2.1; no longer O2.2
- net col4.L: no longer K25.1
- net col5.L: now also K25.1
- net TX-R: now reaches U2.2 (0/PD3)
- net TX-R: now also J2.R2
- net VCC-R: now reaches U2.22 (VCC)
- net VCC-R: now also J2.T
- net GND-R: now reaches U2.24 (GND)
- net GND-R: now also U2.4 (GND), U2.5 (GND), J2.S
- net RX-R: now reaches U2.3 (1/PD2)
- net RX-R: now also J2.R1
- net at D59.2, K62.1: now also O2.2; no longer O2.1
- net TX-L: now reaches U1.2 (0/PD3)
- net TX-L: now also J1.R2
- net VCC-L: now reaches U1.22 (VCC)
- net VCC-L: now also J1.T
- net GND-L: now reaches U1.24 (GND)
- net GND-L: now also U1.4 (GND), U1.5 (GND), J1.S
- net RX-L: now reaches U1.3 (1/PD2)
- net RX-L: now also J1.R1
Other:
- moved on the sheet: D25, K25, O2

Commit message: re-put footprint and newtrack
Connections:
- no-connect marks 0 -> 4
Changed lines of the file:
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@@
 		(color 0 0 0 0)
+	)
+	(no_connect
+		(at 253.365 35.56)
+	)
+	(no_connect
+		(at 35.56 34.925)
+	)
+	(no_connect
+		(at 212.725 35.56)
+	)
+	(no_connect
+		(at 76.2 34.925)
 	)
 	(wire

Commit message: set pinout and layout
Parts:
- added J10, J9: OLED, DreaM117er-keebLibrary:PinHeader_1x04_P2.54mm_Vertical, symbol Connector:Conn_01x04_Pin
- added J3, J4: Left side, DreaM117er-keebLibrary:TRRS-PJ-320A, symbol Connector_Audio:AudioJack4
- added J5, J6: Right side, DreaM117er-keebLibrary:TRRS-PJ-320A, symbol Connector_Audio:AudioJack4
- added J7, J8: Battery PH2.0, Connector_JST:JST_PH_S2B-PH-K_1x02_P2.00mm_Horizontal, symbol Connector:Conn_01x02_Socket
- added SW1: RST-L, DreaM117er-keebLibrary:ResetSW_1side, symbol Switch:SW_Push
- added SW2: RST-R, DreaM117er-keebLibrary:ResetSW_1side, symbol Switch:SW_Push
Connections:
- net GND-L: now also J1.R2, U1.1 (?), J3.R2, J4.R2, J7.2 (Pin_2), J9.4 (Pin_4), SW1.2; no longer J1.S
- net GND-R: now also J2.R2, U2.1 (?), J10.4 (Pin_4), J5.R2, J6.R2, J8.2 (Pin_2), SW2.2; no longer J2.S
- net VCC-L: now also J3.T, J4.T, J9.3 (Pin_3)
- net VCC-R: now also J10.3 (Pin_3), J5.T, J6.T
- net col0.L: now also U1.21 (29/PF4)
- net col0.R: now also U2.21 (29/PF4)
- net col1.L: now also U1.20 (28/PF5)
- net col1.R: now also U2.20 (28/PF5)
- net col2.L: now also U1.19 (27/PF6)
- net col2.R: now also U2.19 (27/PF6)
- net col3.L: now also U1.18 (26/PF7)
- net col3.R: now also U2.18 (26/PF7)
- net col4.L: now also U1.17 (22/PB1)
- net col4.R: now also U2.17 (22/PB1)
- net col5.L: now also U1.16 (20/PB3)
- net col5.R: now also U2.16 (20/PB3)
- net col6.L: now also U1.15 (23/PB2)
- net col6.R: now also U2.15 (23/PB2)
- net col7.R: now also U2.14 (21/PB6)
- net row0: now also U1.9 (5/PC6)
- net row1: now also U1.10 (6/PD7)
- net row2: now also U1.11 (7/PE6)
- net row3: now also U1.12 (8/PB4)
- net row4: now also U1.13 (9/PB5)
- net row5: now also U2.9 (5/PC6)
- net row6: now also U2.10 (6/PD7)
- net row7: now also U2.11 (7/PE6)
- net row8: now also U2.12 (8/PB4)
- net row9: now also U2.13 (9/PB5)
- net RST-R: now reaches U2.23 (RST)
- net RST-R: now also SW2.1
- net BAT+R: now reaches U2.25 (B0)
- net BAT+R: now also U2.26 (?), J8.1 (Pin_1)
- net SDA-R: now reaches U2.6 (2/PD1)
- net SDA-R: now also J10.1 (Pin_1)
- net SCL-R: now reaches U2.7 (3/PD0)
- net SCL-R: now also J10.2 (Pin_2)
- net RST-L: now reaches U1.23 (RST)
- net RST-L: now also SW1.1
- net BAT+L: now reaches U1.25 (B0)
- net BAT+L: now also U1.26 (?), J7.1 (Pin_1)
- net SDA-L: now reaches U1.6 (2/PD1)
- net SDA-L: now also J9.1 (Pin_1)
- net SCL-L: now reaches U1.7 (3/PD0)
- net SCL-L: now also J9.2 (Pin_2)
- net RX-L: no longer names the net of U1.3 (1/PD2)
- net RX-L: no longer J1.R1
- net RX-R: no longer names the net of U2.3 (1/PD2)
- net RX-R: no longer J2.R1
- net TX-L renamed Data-L
- net Data-L: now also J1.R1, J3.R1, J4.R1; no longer J1.R2
- net TX-R renamed Data-R
- net Data-R: now also J2.R1, J5.R1, J6.R1; no longer J2.R2
- no-connect marks 4 -> 11
Other:
- moved on the sheet: J1, J2

Commit message: finish track and zone
Parts:
- added SW3, SW4: ON-OFF, Button_Switch_THT:SW_Slide_SPDT_Angled_CK_OS102011MA1Q, symbol Switch:SW_Reed_SPDT
Connections:
- net BAT+L: now also SW3.2; no longer J7.1 (Pin_1)
- net BAT+R: now also SW4.2; no longer J8.1 (Pin_1)
- new net: J8.1 (Pin_1), SW4.3
- new net: J7.1 (Pin_1), SW3.1
- no-connect marks 11 -> 13
Other:
- moved on the sheet: J7, J8

Commit message: fix TRRS and SlideSW
Parts:
- SW3, SW4: value ON-OFF -> OFF-ON
Connections:
- net GND-L: now also J1.S, J3.S, J4.S; no longer J1.R2, J3.R2, J4.R2
- net GND-R: now also J2.S, J5.S, J6.S; no longer J2.R2, J5.R2, J6.R2
- net at SW4.1: now also J8.1 (Pin_1)
- net at SW4.3: no longer J8.1 (Pin_1)
- net at SW3.1: no longer J7.1 (Pin_1)
- net at SW3.3: now also J7.1 (Pin_1)
Other:
- moved on the sheet: J7, J8
