File: mx66/pcb tiny/6666.kicad_sch (KiCad schematic)
At the start: 145 parts, among them J3 Left side, J5 Right side, K1 100, K10 125, K11 100, K12 100, K13 100, K14 100, K15 125, K16 100, K17 100, K18 100, K19 100, K2 150, K20 125, K21 100, K22 100, K23 100, K24 100, K25 225, K26 100, K27 100, K28 100, K29 100, K3 175, K30 100, K31 100, K32 100, K33 100, K34 100, K35 100, K36 100, K37 100, K38 100, K39 100, K4 225, K40 100, K41 100, K42 100, K43 275, K44 100, K45 100, K46 100, K47 100, K48 125, K49 100, K5 125, K50 100, K51 100, K52 100, K53 125, K54 100, K55 100, K56 100, K57 100, K58 100, K59 100, K6 100, K60 100, K61 100, K62 200, K63 150, K64 225, K65 100, K66 100, K7 100, K8 100, K9 100, U3 MCU_RP2040_SuperMini, U4 MCU_RP2040_SuperMini

Commit message: place footprints
Parts:
- removed J3: Left side, DreaM117er-keebLibrary:TRRS-PJ-320A, symbol Connector_Audio:AudioJack4
- removed J5: Right side, DreaM117er-keebLibrary:TRRS-PJ-320A, symbol Connector_Audio:AudioJack4
- added J1, J2: AudioJack3, DreaM117er-keebLibrary:TRRS-PJ-381-BB_5P, symbol Connector_Audio:AudioJack3
- added JP1: Power, DreaM117er-keebLibrary:Jumper_1-3_SingleSide_Cut, symbol Jumper:Jumper_3_Bridged12
- added JP2: Power, DreaM117er-keebLibrary:Jumper_1-3_SingleSide_Cut2, symbol Jumper:Jumper_3_Bridged12
Connections:
- net Data-L: now also J1.R
- net Data-R: now also J2.R
- net GND-L: now also U3.2 (GND), J1.S
- net GND-R: now also U4.2 (GND), J2.S
- net VCC-L: now also J1.T, JP1.2 (C)
- net VCC-R: now also J2.T, JP2.2 (C)
- net +5V-R: now reaches U4.1 (5V)
- net +5V-R: now also JP2.1 (A)
- net +3V3-R: now reaches U4.3 (3V3)
- net +3V3-R: now also JP2.3 (B)
- net +5V-L: now reaches U3.1 (5V)
- net +5V-L: now also JP1.1 (A)
- net +3V3-L: now reaches U3.3 (3V3)
- net +3V3-L: now also JP1.3 (B)
- no-connect marks 2 -> 0
