File: mx66/pcb v2/6666.kicad_pcb (KiCad board)
At the start: 2 copper layers, 326.7 x 209.2 mm, 115 parts, among them J1 AudioJack3, J2 AudioJack3, J3 AudioJack3, K1 100, K10 125, K100 100, K101 100, K102 150, K103 225, K104 100, K105 100, K11 100, K12 100, K13 100, K14 100, K15 125, K16 100, K17 100, K18 100, K19 100, K2 150, K20 125, K21 100, K22 100, K23 100, K24 100, K25 200, K26 100, K27 100, K28 100, K29 100, K3 175, K30 100, K31 100, K32 100, K33 100, K34 100, K35 100, K36 200, K37 100, K38 100, K39 100, K4 225, K40 100, K41 125, K42 100, K43 100, K44 100, K45 100, K46 100, K47 100, K48 100, K49 100, K5 100, K50 100, K51 100, K52 100, K53 100, K54 100, K55 100, K56 100, K57 100, K58 100, K59 100, K6 100, K60 100, K61 100, K62 100, K63 150, K64 225, K65 275, K66 100, K67 175, K68 100, K69 100, K7 100, K70 100, K71 100, K72 100, K73 100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

Commit message: update new pcb edge
Parts:
- moved K100 41.0 mm to (291.6, 238.6)
- moved K57 41.0 mm to (291.6, 52.4)
- moved K61 41.0 mm to (291.6, 128.6)
- moved K96 41.0 mm to (291.6, 162.3)
- moved K99 41.0 mm to (291.6, 219.5)
- moved K32 41.0 mm to (167.8, 71.4)
- moved K38 41.0 mm to (205.9, 71.4)
- moved K41 41.0 mm to (213.1, 128.6)
- moved K43 41.0 mm to (225.0, 71.4)
- moved K44 41.0 mm to (210.7, 90.5)
- moved K47 41.0 mm to (253.5, 52.4)
- moved K48 41.0 mm to (244.0, 71.4)
- moved K51 41.0 mm to (253.5, 128.6)
- moved K54 41.0 mm to (248.8, 90.5)
- moved K70 41.0 mm to (167.8, 181.4)
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Other:
- board size 326.7 x 209.2 mm -> 285.8 x 211 mm
